File: PCB/EDAMAME_S/EDAMAME_S.sch (KiCad schematic (older format))
At the start: 58 parts, among them CN1 USB-B-MICRO, J1 Conn_01x20, J2 Conn_01x20, J5 Nichrome, J6 Charge, M1 Motor_L, M2 Motor_R, Q1 NDS9936, Q2 FDS4675, Q3 2SC2712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

Commit message: Readme
Parts:
- BT1, BT2, BT3: symbol Battery_Cell -> Device:Battery_Cell
- C1, C10, C11, C12, C13, C14, C2, C3, C4, C5, C6, C7, C8, C9: symbol C_Small -> Device:C_Small
- CN1: symbol USB-B-MICRO -> user_library:USB-B-MICRO
- D1, D2, D6, D7: symbol LED_Small_ALT -> Device:LED_Small_ALT
- D3, D4, D5: symbol D_Small_ALT -> Device:D_Small_ALT
- J1, J2: symbol Conn_01x20 -> conn:Conn_01x20
- J5: symbol Conn_01x02 -> conn:Conn_01x02
- J6: symbol Conn_01x03 -> conn:Conn_01x03
- M1, M2: symbol Motor_DC -> motors:Motor_DC
- Q1: symbol FDS9926A -> transistors:FDS9926A
- Q2: symbol FDS4675 -> user_library:FDS4675
- Q3: symbol Q_NPN_BEC -> Device:Q_NPN_BEC
- R1, R10, R11, R12, R13, R14, R2, R3, R4, R5, R6, R7, R8, R9: symbol R -> Device:R
- SW1: symbol SW_DIP_x01 -> switches:SW_DIP_x01
- U1: symbol microSD -> user_library:microSD
- U2: symbol FT231XS -> ftdi:FT231XS
- U3: symbol ESP32-WROOM -> ESP32-footprints-Shem-Lib:ESP32-WROOM
- U4: symbol L7805 -> regul:L7805
- U5: symbol LSM303C -> user_library:LSM303C
- U6: symbol GPS-54D -> user_library:GPS-54D
- U7, U9: symbol BD6231F_2 -> user_library:BD6231F_2
- U8: symbol INA226 -> user_library:INA226
Connections:
- wire segments 250 -> 322
