File: PCB/EDAMAME_S/EDAMAME_S.sch (KiCad schematic (older format))
At the start: 58 parts, among them CN1 USB-B-MICRO, J1 Conn_01x20, J2 Conn_01x20, J5 Nichrome, J6 Charge, M1 Motor_L, M2 Motor_R, Q1 NDS9936, Q2 FDS4675, Q3 2SC2712, SW1 power, U1 microSD, U2 FT231XS, U3 ESP32-WROOM, U4 NJM2391DL1-33, U5 LSM303C, U6 GPS-54D, U7 BD6231F, U8 INA226, U9 BD6231F

Commit message: 回路変更(フットプリントの割り当てはまだ）
Parts:
- removed BT2: 10440, user:BH-411, symbol Device:Battery_Cell
- removed J6: Charge, EH:S3B-EH, symbol conn:Conn_01x03
- removed Q1: NDS9936, Housings_SOIC:SOIC-8_3.9x4.9mm_Pitch1.27mm, symbol transistors:FDS9926A
- removed U4: NJM2391DL1-33, TO_SOT_Packages_SMD:TO-252-2_Rectifier, symbol regul:L7805
- removed U6: GPS-54D, user:GPS-54, symbol user_library:GPS-54D
- added C15, C16: 10u, Capacitor_SMD:C_0805_2012Metric_Pad1.15x1.40mm_HandSolder, symbol Device:C_Small
- added D8: GPS, LED_SMD:LED_0603_1608Metric_Pad1.05x0.95mm_HandSolder, symbol Device:LED_Small_ALT
- added L1: 2.2uH VLF4012-2R2, symbol Device:L
- added Q1: 2N7002DW, Package_TO_SOT_SMD:SOT-363_SC-70-6_Handsoldering, symbol user_library:2N7002DW
- added R15: 1K, Resistor_SMD:R_0603_1608Metric_Pad1.05x0.95mm_HandSolder, symbol Device:R
- added SW2: RST, user:SKRPACE010_kai, symbol Switch:SW_Push
- added U4: TPS63000, Package_SON:Texas_S-PWSON-N10_ThermalVias, symbol user_library:TPS63000
- added U6: GYSFDMAXB, symbol user_library:GYSFDMAXB
- C1, C12, C2, C3, C4, C5, C6, C7, C8, C9: footprint Capacitors_SMD:C_0603_HandSoldering -> Capacitor_SMD:C_0603_1608Metric_Pad1.05x0.95mm_HandSolder
- C10: footprint Capacitors_SMD:C_1206_HandSoldering -> Capacitor_SMD:C_1210_3225Metric_Pad1.42x2.65mm_HandSolder
- C11, C13: footprint Capacitors_SMD:C_1206_HandSoldering -> Capacitor_SMD:C_0805_2012Metric_Pad1.15x1.40mm_HandSolder
- C14: value 10u -> 0.1u; footprint Capacitors_SMD:C_0603_HandSoldering -> Capacitor_SMD:C_0603_1608Metric_Pad1.05x0.95mm_HandSolder
- D1, D2, D6, D7: footprint LEDs:LED_0603_HandSoldering -> LED_SMD:LED_0603_1608Metric_Pad1.05x0.95mm_HandSolder
- D3, D4, D5: footprint Diodes_SMD:D_SOD-123F -> Diode_SMD:D_SOD-123F
- J1, J2: footprint Socket_Strips:Socket_Strip_Straight_1x20_Pitch2.54mm -> Connector_PinHeader_2.54mm:PinHeader_1x20_P2.54mm_Vertical
- M1, M2: footprint EH:B2B-EH -> Connector_JST:JST_XH_B02B-XH-A_1x02_P2.50mm_Vertical
- Q2: footprint Housings_SOIC:SOIC-8_3.9x4.9mm_Pitch1.27mm -> Package_SO:SOIC-8_3.9x4.9mm_P1.27mm
- Q3: footprint TO_SOT_Packages_SMD:SOT-23_Handsoldering -> Package_TO_SOT_SMD:SOT-23_Handsoldering
- R1, R10, R11, R13, R14, R2, R3, R4, R5, R6, R7, R8, R9: footprint Resistors_SMD:R_0603_HandSoldering -> Resistor_SMD:R_0603_1608Metric_Pad1.05x0.95mm_HandSolder
- R12: footprint Resistors_SMD:R_2512_HandSoldering -> Resistor_SMD:R_2512_6332Metric_Pad1.52x3.35mm_HandSolder
- U2: footprint SMD_Packages:SSOP-20 -> Package_SO:SSOP-20_4.4x6.5mm_P0.65mm
- U7, U9: value BD6231F -> BD6211F
Connections:
- wire segments 322 -> 348

Commit message: フットプリント割当
Parts:
- CN1: footprint mylib:Micro-USB -> user:Micro-USB
- L1: footprint (none) -> user:inductor_VLF4012-2R2
- SW1: footprint mylib:SS-12D01-VG4 -> user:SS-12D01-VG4
- U2: footprint Package_SO:SSOP-20_4.4x6.5mm_P0.65mm -> user:FT231XS
- U6: footprint (none) -> user:GYSFDMAXB
Changed lines of the file:
@@
 F 0 "U2" H 2150 2550 50  0000 L CNN
 F 1 "FT231XS" H 3000 2550 50  0000 L CNN
-F 2 "Package_SO:SSOP-20_4.4x6.5mm_P0.65mm" H 2700 1750 50  0001 C CNN
+F 2 "user:FT231XS" H 2700 1750 50  0001 C CNN
 F 3 "" H 2700 1750 50  0001 C CNN
 	1    2700 1750
@@
 F 0 "SW1" H 1250 6100 50  0000 C CNN
 F 1 "power" H 1250 5800 50  0000 C CNN
-F 2 "mylib:SS-12D01-VG4" H 1250 5950 50  0001 C CNN
+F 2 "user:SS-12D01-VG4" H 1250 5950 50  0001 C CNN
 F 3 "" H 1250 5950 50  0001 C CNN
 	1    1250 5950
@@
 F 0 "CN1" H 850 1850 60  0000 C CNN
 F 1 "USB-B-MICRO" H 1000 1950 60  0000 C CNN
-F 2 "mylib:Micro-USB" H 1000 1550 60  0001 C CNN
+F 2 "user:Micro-USB" H 1000 1550 60  0001 C CNN
 F 3 "" H 1000 1550 60  0000 C CNN
 	1    1000 1550
@@
 F 0 "L1" V 2440 3250 50  0000 C CNN
 F 1 "2.2uH VLF4012-2R2" V 2349 3250 50  0000 C CNN
-F 2 "" H 2250 3250 50  0001 C CNN
+F 2 "user:inductor_VLF4012-2R2" H 2250 3250 50  0001 C CNN
 F 3 "~" H 2250 3250 50  0001 C CNN
 	1    2250 3250
@@
 F 0 "U6" H 8050 3300 60  0000 C CNN
 F 1 "GYSFDMAXB" H 8050 3400 60  0000 C CNN
-F 2 "" H 7600 4450 60  0001 C CNN
+F 2 "user:GYSFDMAXB" H 7600 4450 60  0001 C CNN
 F 3 "" H 7600 4450 60  0001 C CNN
 	1    8300 4450

Commit message: 回路図AVRに変更
Parts:
- removed BT1: BACKUP, user:MS621FE_FL11E, symbol Device:Battery_Cell
- removed BT3: 10440, user:BH-411, symbol Device:Battery_Cell
- removed C1, C12, C14, C2, C5, C7, C8, C9: 0.1u, Capacitor_SMD:C_0603_1608Metric_Pad1.05x0.95mm_HandSolder, symbol Device:C_Small
- removed C10: 100u, Capacitor_SMD:C_1210_3225Metric_Pad1.42x2.65mm_HandSolder, symbol Device:C_Small
- removed C11, C13, C15, C16: 10u, Capacitor_SMD:C_0805_2012Metric_Pad1.15x1.40mm_HandSolder, symbol Device:C_Small
- removed C3, C4: 47p, Capacitor_SMD:C_0603_1608Metric_Pad1.05x0.95mm_HandSolder, symbol Device:C_Small
- removed C6: 10u, Capacitor_SMD:C_0603_1608Metric_Pad1.05x0.95mm_HandSolder, symbol Device:C_Small
- removed CN1: USB-B-MICRO, user:Micro-USB, symbol user_library:USB-B-MICRO
- removed D1: TXLED, LED_SMD:LED_0603_1608Metric_Pad1.05x0.95mm_HandSolder, symbol Device:LED_Small_ALT
- removed D2: RXLED, LED_SMD:LED_0603_1608Metric_Pad1.05x0.95mm_HandSolder, symbol Device:LED_Small_ALT
- removed D3, D4, D5: GS1010FL, Diode_SMD:D_SOD-123F, symbol Device:D_Small_ALT
- removed D6: Nichrome, LED_SMD:LED_0603_1608Metric_Pad1.05x0.95mm_HandSolder, symbol Device:LED_Small_ALT
- removed D7: POWER, LED_SMD:LED_0603_1608Metric_Pad1.05x0.95mm_HandSolder, symbol Device:LED_Small_ALT
- removed D8: GPS, LED_SMD:LED_0603_1608Metric_Pad1.05x0.95mm_HandSolder, symbol Device:LED_Small_ALT
- removed J1, J2: Conn_01x20, Connector_PinHeader_2.54mm:PinHeader_1x20_P2.54mm_Vertical, symbol conn:Conn_01x20
- removed J5: Nichrome, user:MPT0.5_2-2.54, symbol conn:Conn_01x02
- removed L1: 2.2uH VLF4012-2R2, user:inductor_VLF4012-2R2, symbol Device:L
- removed M1: Motor_L, Connector_JST:JST_XH_B02B-XH-A_1x02_P2.50mm_Vertical, symbol motors:Motor_DC
- removed M2: Motor_R, Connector_JST:JST_XH_B02B-XH-A_1x02_P2.50mm_Vertical, symbol motors:Motor_DC
- removed Q1: 2N7002DW, Package_TO_SOT_SMD:SOT-363_SC-70-6_Handsoldering, symbol user_library:2N7002DW
- removed Q2: FDS4675, Package_SO:SOIC-8_3.9x4.9mm_P1.27mm, symbol user_library:FDS4675
- removed Q3: 2SC2712, Package_TO_SOT_SMD:SOT-23_Handsoldering, symbol Device:Q_NPN_BEC
- removed R1, R11, R14, R9: 10K, Resistor_SMD:R_0603_1608Metric_Pad1.05x0.95mm_HandSolder, symbol Device:R
- removed R10, R13, R15, R4, R5: 1K, Resistor_SMD:R_0603_1608Metric_Pad1.05x0.95mm_HandSolder, symbol Device:R
- removed R12: 10m, Resistor_SMD:R_2512_6332Metric_Pad1.52x3.35mm_HandSolder, symbol Device:R
- removed R2, R3: 33, Resistor_SMD:R_0603_1608Metric_Pad1.05x0.95mm_HandSolder, symbol Device:R
- removed R6, R7: 2.2K, Resistor_SMD:R_0603_1608Metric_Pad1.05x0.95mm_HandSolder, symbol Device:R
- removed R8: 100, Resistor_SMD:R_0603_1608Metric_Pad1.05x0.95mm_HandSolder, symbol Device:R
- removed SW1: power, user:SS-12D01-VG4, symbol switches:SW_DIP_x01
- removed SW2: RST, user:SKRPACE010_kai, symbol Switch:SW_Push
- removed U1: microSD, user:microSD, symbol user_library:microSD
- removed U2: FT231XS, user:FT231XS, symbol ftdi:FT231XS
- removed U3: ESP32-WROOM, ESP32-footprints-Lib:ESP32-WROOM, symbol ESP32-footprints-Shem-Lib:ESP32-WROOM
- removed U4: TPS63000, Package_SON:Texas_S-PWSON-N10_ThermalVias, symbol user_library:TPS63000
- removed U5: LSM303C, Housings_LGA:LGA-12_2x2mm_Pitch0.5mm, symbol user_library:LSM303C
- removed U6: GYSFDMAXB, user:GYSFDMAXB, symbol user_library:GYSFDMAXB
- removed U7, U9: BD6211F, Housings_SOIC:SOIC-8_3.9x4.9mm_Pitch1.27mm, symbol user_library:BD6231F_2
- removed U8: INA226, Housings_SSOP:MSOP-10_3x3mm_Pitch0.5mm, symbol user_library:INA226
Connections:
- net labels removed: +3.3V, +5V, +BATT, BOOT, DTR, EN, ESP32→GPS, ESP32→PC, GND, GNDPWR, GPS→ESP32, I2C_SCL, I2C_SDA, IO13, IO14, IO25, IO26, IO27, IO32, IO33, IO34, IO35, MOTOR_LF, MOTOR_LR, MOTOR_RF, MOTOR_RR, Nichrome, PC→ESP32, RST, SCL, SDA, SPI_CS, SPI_MISO, SPI_MOSI, SPI_SCLK, S_VN, S_VP, VCC, VDC
- wire segments 348 -> 0
- no-connect marks 26 -> 0

Commit message: EdamameS_V1.10
Parts:
- added BT1: BACKUP, user:MS621FE_FL11E, symbol Device:Battery_Cell
- added BT2, BT3: 10440, user:BH-411, symbol Device:Battery_Cell
- added C1, C12, C2, C5, C7, C8, C9: 0.1u, Capacitors_SMD:C_0603_HandSoldering, symbol Device:C_Small
- added C10: 100u, Capacitors_SMD:C_1206_HandSoldering, symbol Device:C_Small
- added C11, C13: 10u, Capacitors_SMD:C_1206_HandSoldering, symbol Device:C_Small
- added C14, C6: 10u, Capacitors_SMD:C_0603_HandSoldering, symbol Device:C_Small
- added C3, C4: 47p, Capacitors_SMD:C_0603_HandSoldering, symbol Device:C_Small
- added CN1: USB-B-MICRO, mylib:Micro-USB, symbol user_library:USB-B-MICRO
- added D1: TXLED, LEDs:LED_0603_HandSoldering, symbol Device:LED_Small_ALT
- added D2: RXLED, LEDs:LED_0603_HandSoldering, symbol Device:LED_Small_ALT
- added D3, D4, D5: GS1010FL, Diodes_SMD:D_SOD-123F, symbol Device:D_Small_ALT
- added D6: Nichrome, LEDs:LED_0603_HandSoldering, symbol Device:LED_Small_ALT
- added D7: POWER, LEDs:LED_0603_HandSoldering, symbol Device:LED_Small_ALT
- added J1, J2: Conn_01x20, Socket_Strips:Socket_Strip_Straight_1x20_Pitch2.54mm, symbol conn:Conn_01x20
- added J5: Nichrome, user:MPT0.5_2-2.54, symbol conn:Conn_01x02
- added J6: Charge, EH:S3B-EH, symbol conn:Conn_01x03
- added M1: Motor_L, EH:B2B-EH, symbol motors:Motor_DC
- added M2: Motor_R, EH:B2B-EH, symbol motors:Motor_DC
- added Q1: NDS9936, Housings_SOIC:SOIC-8_3.9x4.9mm_Pitch1.27mm, symbol transistors:FDS9926A
- added Q2: FDS4675, Housings_SOIC:SOIC-8_3.9x4.9mm_Pitch1.27mm, symbol user_library:FDS4675
- added Q3: 2SC2712, TO_SOT_Packages_SMD:SOT-23_Handsoldering, symbol Device:Q_NPN_BEC
- added R1, R11, R14, R9: 10K, Resistors_SMD:R_0603_HandSoldering, symbol Device:R
- added R10, R13, R4, R5: 1K, Resistors_SMD:R_0603_HandSoldering, symbol Device:R
- added R12: 10m, Resistors_SMD:R_2512_HandSoldering, symbol Device:R
- added R2, R3: 33, Resistors_SMD:R_0603_HandSoldering, symbol Device:R
- added R6, R7: 2.2K, Resistors_SMD:R_0603_HandSoldering, symbol Device:R
- added R8: 100, Resistors_SMD:R_0603_HandSoldering, symbol Device:R
- added SW1: power, mylib:SS-12D01-VG4, symbol switches:SW_DIP_x01
- added U1: microSD, user:microSD, symbol user_library:microSD
- added U2: FT231XS, SMD_Packages:SSOP-20, symbol ftdi:FT231XS
- added U3: ESP32-WROOM, ESP32-footprints-Lib:ESP32-WROOM, symbol ESP32-footprints-Shem-Lib:ESP32-WROOM
- added U4: NJM2391DL1-33, TO_SOT_Packages_SMD:TO-252-2_Rectifier, symbol regul:L7805
- added U5: LSM303C, Housings_LGA:LGA-12_2x2mm_Pitch0.5mm, symbol user_library:LSM303C
- added U6: GPS-54D, user:GPS-54, symbol user_library:GPS-54D
- added U7, U9: BD6231F, Housings_SOIC:SOIC-8_3.9x4.9mm_Pitch1.27mm, symbol user_library:BD6231F_2
- added U8: INA226, Housings_SSOP:MSOP-10_3x3mm_Pitch0.5mm, symbol user_library:INA226
Connections:
- net labels added: +3.3V, +5V, +BATT, BOOT, DTR, EN, ESP32→GPS, ESP32→PC, GND, GNDPWR, GPS→ESP32, I2C_SCL, I2C_SDA, IO13, IO14, IO25, IO26, IO27, IO32, IO33, IO34, IO35, MOTOR_LF, MOTOR_LR, MOTOR_RF, MOTOR_RR, Nichrome, PC→ESP32, RST, SCL, SDA, SPI_CS, SPI_MISO, SPI_MOSI, SPI_SCLK, S_VN, S_VP, VCC, VDC
- wire segments 0 -> 322
- no-connect marks 0 -> 26
