File: PCB/EDAMAME_S/EDAMAME_S.kicad_pcb (KiCad board)
At the start: 2 copper layers, 80 x 87 mm, 60 parts, among them CN1 USB-B-MICRO, J1 Conn_01x20, J2 Conn_01x20, J5 Nichrome, J6 CHARGE, M1 Motor_L, M2 Motor_R, Q1 NDS9936, Q2 FDS4675, Q3 2SC2712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

Commit message: フットプリント割当
Parts:
- removed BT2: 10440, user:BH-411
- removed G*** (x2): LOGO, mod:SOMESAT_LOGO
- removed J6: CHARGE, EH:S3B-EH
- added C15: 10u, Capacitor_SMD:C_0805_2012Metric_Pad1.15x1.40mm_HandSolder, F.Cu at (64.1, 6.64)
- added C16: 10u, Capacitor_SMD:C_0805_2012Metric_Pad1.15x1.40mm_HandSolder, F.Cu at (69.8, 6.54)
- added D8: GPS, LED_SMD:LED_0603_1608Metric_Pad1.05x0.95mm_HandSolder, F.Cu at (67.7, 8.31)
- added L1: 2.2uH VLF4012-2R2, user:inductor_VLF4012-2R2, F.Cu at (70.3, 3.74)
- added R15: 1K, Resistor_SMD:R_0603_1608Metric_Pad1.05x0.95mm_HandSolder, F.Cu at (63.9, 8.37)
- added SW2: RST, user:SKRPACE010_kai, F.Cu at (65.1, 3.79)
- C1, C12, C2, C3, C4, C5, C6, C7, C8, C9: footprint Capacitors_SMD:C_0603_HandSoldering -> Capacitor_SMD:C_0603_1608Metric_Pad1.05x0.95mm_HandSolder
- C10: footprint Capacitors_SMD:C_1206_HandSoldering -> Capacitor_SMD:C_1210_3225Metric_Pad1.42x2.65mm_HandSolder
- C11, C13: footprint Capacitors_SMD:C_1206_HandSoldering -> Capacitor_SMD:C_0805_2012Metric_Pad1.15x1.40mm_HandSolder
- C14: value 10u -> 0.1u; footprint Capacitors_SMD:C_0603_HandSoldering -> Capacitor_SMD:C_0603_1608Metric_Pad1.05x0.95mm_HandSolder
- CN1: footprint mylib:Micro-USB -> user:Micro-USB
- D1, D2, D6, D7: footprint LEDs:LED_0603_HandSoldering -> LED_SMD:LED_0603_1608Metric_Pad1.05x0.95mm_HandSolder
- D3, D4, D5: footprint Diodes_SMD:D_SOD-123F -> Diode_SMD:D_SOD-123F
- J1, J2: footprint Socket_Strips:Socket_Strip_Straight_1x20_Pitch2.54mm -> Connector_PinHeader_2.54mm:PinHeader_1x20_P2.54mm_Vertical
- M1, M2: footprint EH:B2B-EH -> Connector_JST:JST_XH_B02B-XH-A_1x02_P2.50mm_Vertical
- Q1: value NDS9936 -> 2N7002DW; footprint Housings_SOIC:SOIC-8_3.9x4.9mm_Pitch1.27mm -> Package_TO_SOT_SMD:SOT-363_SC-70-6_Handsoldering
- Q2: footprint Housings_SOIC:SOIC-8_3.9x4.9mm_Pitch1.27mm -> Package_SO:SOIC-8_3.9x4.9mm_P1.27mm
- Q3: footprint TO_SOT_Packages_SMD:SOT-23_Handsoldering -> Package_TO_SOT_SMD:SOT-23_Handsoldering
- R1, R10, R11, R13, R14, R2, R3, R4, R5, R6, R7, R8, R9: footprint Resistors_SMD:R_0603_HandSoldering -> Resistor_SMD:R_0603_1608Metric_Pad1.05x0.95mm_HandSolder
- R12: footprint Resistors_SMD:R_2512_HandSoldering -> Resistor_SMD:R_2512_6332Metric_Pad1.52x3.35mm_HandSolder
- SW1: footprint mylib:SS-12D01-VG4 -> user:SS-12D01-VG4
- U2: footprint SMD_Packages:SSOP-20 -> user:FT231XS
- U4: value NJM2391DL1-33 -> TPS63000; footprint TO_SOT_Packages_SMD:TO-252-2_Rectifier -> Package_SON:Texas_S-PWSON-N10_ThermalVias
- U6: value GPS-54D -> GYSFDMAXB; footprint user:GPS-54 -> user:GYSFDMAXB
- U7, U9: value BD6231F -> BD6211F
Connections:
- BT3 pad 1: Net-(BT2-Pad2) -> Net-(BT3-Pad1)
- C9 pad 1: Net-(C9-Pad1) -> Net-(C15-Pad1)
- CN1 pad 4: (no net) -> Net-(CN1-Pad4)
- D3 pad 1: Net-(C9-Pad1) -> Net-(C15-Pad1)
- D4 pad 1: Net-(C9-Pad1) -> Net-(C15-Pad1)
- J2 pad 10: (no net) -> Net-(J2-Pad10)
- J2 pad 11: (no net) -> Net-(J2-Pad11)
- J2 pad 12: (no net) -> Net-(J2-Pad12)
- J2 pad 7: (no net) -> Net-(J2-Pad7)
- J2 pad 8: (no net) -> Net-(J2-Pad8)
- J2 pad 9: (no net) -> Net-(J2-Pad9)
- Q1 pad 1: /DTR -> /RST
- Q1 pad 2: /RST -> /DTR
- Q1 pad 3: /RST -> /BOOT
- Q1 pad 5: /EN -> /RST
- SW1 pad 2: Net-(BT2-Pad1) -> Net-(BT3-Pad1)
- U1 pad 1: (no net) -> Net-(U1-Pad1)
- U1 pad 8: (no net) -> Net-(U1-Pad8)
- U2 pad 13: (no net) -> Net-(U2-Pad13)
- U2 pad 18: (no net) -> Net-(U2-Pad18)
- U2 pad 19: (no net) -> Net-(U2-Pad19)
- U2 pad 5: (no net) -> Net-(U2-Pad5)
- U2 pad 7: (no net) -> Net-(U2-Pad7)
- U2 pad 8: (no net) -> Net-(U2-Pad8)
- U2 pad 9: (no net) -> Net-(U2-Pad9)
- U3 pad 17: (no net) -> Net-(U3-Pad17)
- U3 pad 18: (no net) -> Net-(U3-Pad18)
- U3 pad 19: (no net) -> Net-(U3-Pad19)
- U3 pad 2: +3V3 -> Net-(U3-Pad2)
- U3 pad 20: (no net) -> Net-(U3-Pad20)
- U3 pad 21: (no net) -> Net-(U3-Pad21)
- U3 pad 22: (no net) -> Net-(U3-Pad22)
- U3 pad 24: (no net) -> Net-(U3-Pad24)
- U3 pad 32: (no net) -> Net-(U3-Pad32)
- U4 pad 1: Net-(C9-Pad1) -> +3V3
- U4 pad 2: GND -> Net-(L1-Pad2)
- U4 pad 3: +3V3 -> GND
- U5 pad 11: (no net) -> Net-(U5-Pad11)
- U5 pad 12: (no net) -> Net-(U5-Pad12)
- U5 pad 7: (no net) -> Net-(U5-Pad7)
- U6 pad 1: /ESP32→GPS -> GND
- U6 pad 3: /GPS→ESP32 -> /ESP32→GPS
- U6 pad 4: Net-(BT1-Pad1) -> Net-(U6-Pad4)
- U6 pad 5: +3V3 -> /GPS→ESP32
- U6 pad 6: (no net) -> Net-(R15-Pad1)
- U6 pad 7: (no net) -> GND
- U6 pad 8: (no net) -> Net-(U6-Pad8)
- U8 pad 3: (no net) -> Net-(U8-Pad3)
Routing:
- net Net-(BT3-Pad1): track 0.00 -> 83.6 mm
- net Net-(BT2-Pad2): track 65.7 -> 0.00 mm
- net Net-(BT2-Pad1): track 31.3 -> 13.5 mm
- net Net-(C9-Pad1): track 8.38 -> 0.00 mm
- net Net-(C15-Pad1): track 0.00 -> 8.38 mm
