File: PCB/EDAMAME_S/EDAMAME_S_Ex.sch (KiCad schematic (older format))
At the start: 21 parts, among them J3 Conn, J4 Nichrome, M1 Motor_L, M2 Motor_R, Q1 FDS4675, Q2 2SC2712, SW1 power, U7 BD6211F, U8 INA226, U9 BD6211F

Commit message: AVR フットプリント・基板外形割当
Parts:
- removed Q1: FDS4675, Package_SO:SOIC-8_3.9x4.9mm_P1.27mm, symbol user_library:FDS4675
- added Q1: MTM231102LBF, Package_TO_SOT_SMD:SOT-323_SC-70_Handsoldering, symbol Device:Q_PMOS_GSD
- J4: footprint TerminalBlock:TerminalBlock_bornier-2_P5.08mm -> user:MPT0.5_2-2.54; 品番 (none) -> P-08450; 購入先 (none) -> 秋月
Connections:
- wire segments 100 -> 89
Changed lines of the file:
@@
 L Device:Q_NPN_BEC Q2
 U 1 1 5B1D0A0A
-P 4900 3250
-F 0 "Q2" H 5100 3300 50  0000 L CNN
-F 1 "2SC2712" H 5100 3200 50  0000 L CNN
-F 2 "Package_TO_SOT_SMD:SOT-23_Handsoldering" H 5100 3350 50  0001 C CNN
-F 3 "" H 4900 3250 50  0001 C CNN
-	1    4900 3250
-	1    0    0    -1
-$EndComp
-$Comp
-L user_library:FDS4675 Q1
-U 1 1 5B1D0AAB
-P 5850 2650
-F 0 "Q1" H 5450 3100 50  0000 L CNN
-F 1 "FDS4675" H 5350 2500 50  0000 L CNN
-F 2 "Package_SO:SOIC-8_3.9x4.9mm_P1.27mm" H 5350 2900 50  0001 C CNN
-F 3 "" H 5550 2800 50  0001 C CNN
-	1    5850 2650
-	-1   0    0    1
+P 5450 2950
+F 0 "Q2" H 5650 3000 50  0000 L CNN
+F 1 "2SC2712" H 5650 2900 50  0000 L CNN
+F 2 "Package_TO_SOT_SMD:SOT-23_Handsoldering" H 5650 3050 50  0001 C CNN
+F 3 "" H 5450 2950 50  0001 C CNN
+	1    5450 2950
+	1    0    0    -1
 $EndComp
 $Comp
@@
 Text Label 4500 5850 0    60   ~ 0
 MOTOR_RR
-Text Label 3900 3250 0    60   ~ 0
+Text Label 4450 2950 0    60   ~ 0
 Nichrome
 $Comp
@@
 L Device:R R19
 U 1 1 5B1F2A00
-P 4450 3250
-F 0 "R19" V 4350 3250 50  0000 C CNN
-F 1 "10K" V 4450 3250 50  0000 C CNN
-F 2 "Resistor_SMD:R_0603_1608Metric_Pad1.05x0.95mm_HandSolder" V 4380 3250 50  0001 C CNN
-F 3 "" H 4450 3250 50  0001 C CNN
-	1    4450 3250
+P 5000 2950
+F 0 "R19" V 4900 2950 50  0000 C CNN
+F 1 "10K" V 5000 2950 50  0000 C CNN
+F 2 "Resistor_SMD:R_0603_1608Metric_Pad1.05x0.95mm_HandSolder" V 4930 2950 50  0001 C CNN
+F 3 "" H 5000 2950 50  0001 C CNN
+	1    5000 2950
 	0    1    1    0
 $EndComp
@@
 L Device:R R17
 U 1 1 5B1F308A
-P 5000 2700
-F 0 "R17" V 4900 2700 50  0000 C CNN
-F 1 "10K" V 5000 2700 50  0000 C CNN
-F 2 "Resistor_SMD:R_0603_1608Metric_Pad1.05x0.95mm_HandSolder" V 4930 2700 50  0001 C CNN
-F 3 "" H 5000 2700 50  0001 C CNN
-	1    5000 2700
+P 5550 2400
+F 0 "R17" V 5450 2400 50  0000 C CNN
+F 1 "10K" V 5550 2400 50  0000 C CNN
+F 2 "Resistor_SMD:R_0603_1608Metric_Pad1.05x0.95mm_HandSolder" V 5480 2400 50  0001 C CNN
+F 3 "" H 5550 2400 50  0001 C CNN
+	1    5550 2400
 	-1   0    0    1
 $EndComp
@@
 L power:+BATT #PWR0146
 U 1 1 5B1F4B60
-P 5000 2450
-F 0 "#PWR0146" H 5000 2300 50  0001 C CNN
-F 1 "+BATT" H 5000 2590 50  0000 C CNN
-F 2 "" H 5000 2450 50  0001 C CNN
-F 3 "" H 5000 2450 50  0001 C CNN
-	1    5000 2450
+P 5550 2150
+F 0 "#PWR0146" H 5550 2000 50  0001 C CNN
+F 1 "+BATT" H 5550 2290 50  0000 C CNN
+F 2 "" H 5550 2150 50  0001 C CNN
+F 3 "" H 5550 2150 50  0001 C CNN
+	1    5550 2150
 	1    0    0    -1
 $EndComp
@@
 L power:+BATT #PWR0147
 U 1 1 5B1F4BDD
-P 5650 2450
-F 0 "#PWR0147" H 5650 2300 50  0001 C CNN
-F 1 "+BATT" H 5650 2590 50  0000 C CNN
-F 2 "" H 5650 2450 50  0001 C CNN
-F 3 "" H 5650 2450 50  0001 C CNN
-	1    5650 2450
+P 6700 2050
+F 0 "#PWR0147" H 6700 1900 50  0001 C CNN
+F 1 "+BATT" H 6700 2190 50  0000 C CNN
+F 2 "" H 6700 2050 50  0001 C CNN
+F 3 "" H 6700 2050 50  0001 C CNN
+	1    6700 2050
 	1    0    0    -1
 $EndComp
@@
 F 0 "J4" H 7250 3500 50  0000 C CNN
 F 1 "Nichrome" V 7350 3400 50  0000 C CNN
-F 2 "TerminalBlock:TerminalBlock_bornier-2_P5.08mm" H 7250 3400 50  0001 C CNN
-F 3 "" H 7250 3400 50  0001 C CNN
+F 2 "user:MPT0.5_2-2.54" H 7250 3400 50  0001 C CNN
+F 3 "http://akizukidenshi.com/catalog/g/gP-08450/" H 7250 3400 50  0001 C CNN
+F 4 "P-08450" H 0   0   50  0001 C CNN "品番"
+F 5 "秋月" H 0   0   50  0001 C CNN "購入先"
 	1    7250 3400
 	1    0    0    -1
@@
 L EDAMAME_S-rescue:GNDPWR #PWR0155
 U 1 1 5B2265D9
-P 5000 3450
-F 0 "#PWR0155" H 5000 3250 50  0001 C CNN
-F 1 "GNDPWR" H 5000 3300 50  0000 C CNN
-F 2 "" H 5000 3400 50  0001 C CNN
-F 3 "" H 5000 3400 50  0001 C CNN
-	1    5000 3450
+P 5550 3150
+F 0 "#PWR0155" H 5550 2950 50  0001 C CNN
+F 1 "GNDPWR" H 5550 3000 50  0000 C CNN
+F 2 "" H 5550 3100 50  0001 C CNN
+F 3 "" H 5550 3100 50  0001 C CNN
+	1    5550 3150
 	1    0    0    -1
 $EndComp
@@
 Wire Wire Line
 	7050 3750 7050 3500
-Connection ~ 6700 2750
-Wire Wire Line
-	6550 2650 6700 2650
-Connection ~ 6700 2850
-Wire Wire Line
-	6700 2750 6550 2750
-Wire Wire Line
-	6550 2850 6700 2850
-Connection ~ 6700 2950
-Wire Wire Line
-	6700 2650 6700 2750
 Wire Wire Line
 	7050 2950 7050 3400
 Wire Wire Line
-	6550 2950 6700 2950
-Wire Wire Line
 	6700 3300 6700 3400
 Wire Wire Line
 	6700 3750 6700 3600
-Connection ~ 5650 2650
-Wire Wire Line
-	5850 2650 5650 2650
-Connection ~ 5650 2750
-Wire Wire Line
-	5850 2750 5650 2750
-Wire Wire Line
-	5650 2850 5850 2850
-Wire Wire Line
-	5650 2450 5650 2650
-Wire Wire Line
-	5000 2550 5000 2450
-Connection ~ 5000 2950
-Wire Wire Line
-	5000 2950 5850 2950
-Wire Wire Line
-	5000 2850 5000 2950
-Wire Wire Line
-	4600 3250 4700 3250
+Wire Wire Line
+	5550 2250 5550 2150
+Connection ~ 5550 2650
+Wire Wire Line
+	5550 2650 6400 2650
+Wire Wire Line
+	5550 2550 5550 2650
+Wire Wire Line
+	5150 2950 5250 2950
 Wire Wire Line
 	6500 6000 6750 6000
@@
 Connection ~ 5700 4200
 Wire Wire Line
-	3900 3250 4300 3250
+	4450 2950 4850 2950
 Wire Wire Line
 	4500 4600 5000 4600
@@
 	2800 4550 2800 4850
 Wire Wire Line
-	6700 2750 6700 2850
-Wire Wire Line
-	6700 2850 6700 2950
-Wire Wire Line
 	6700 2950 7050 2950
 Wire Wire Line
 	6700 2950 6700 3000
 Wire Wire Line
-	5650 2650 5650 2750
-Wire Wire Line
-	5650 2750 5650 2850
-Wire Wire Line
-	5000 2950 5000 3050
+	5550 2650 5550 2750
 Wire Wire Line
 	5500 5350 5700 5350
@@
 Wire Wire Line
 	2650 2100 2050 2100
+Wire Wire Line
+	6700 2050 6700 2450
+$Comp
+L Device:Q_PMOS_GSD Q1
+U 1 1 5C1A7D47
+P 6600 2650
+F 0 "Q1" H 6806 2696 50  0000 L CNN
+F 1 "MTM231102LBF" H 6806 2605 50  0000 L CNN
+F 2 "Package_TO_SOT_SMD:SOT-323_SC-70_Handsoldering" H 6800 2750 50  0001 C CNN
+F 3 "~" H 6600 2650 50  0001 C CNN
+F 4 " 787-7526" H 0   0   50  0001 C CNN "品番"
+F 5 "RS" H 0   0   50  0001 C CNN "購入先"
+	1    6600 2650
+	1    0    0    -1
+$EndComp
+Wire Wire Line
+	6700 2950 6700 2850
+Connection ~ 6700 2950
 $EndSCHEMATC

Commit message: えだまめS 基板更新
Parts:
- added C20, C21: 0.1u, Capacitor_SMD:C_0603_1608Metric_Pad1.05x0.95mm_HandSolder, symbol Device:C_Small
- added U10: LSM303C, user:LGA-12_2x2mm_P0.5mm_HandSolder, symbol Sensor_Motion:LSM303C
- Q1: footprint Package_TO_SOT_SMD:SOT-323_SC-70_Handsoldering -> Package_TO_SOT_SMD:SOT-323_SC-70
- Q2: footprint Package_TO_SOT_SMD:SOT-23_Handsoldering -> Package_TO_SOT_SMD:SOT-23
Connections:
- wire segments 89 -> 110

Commit message: Add flightpin
Parts:
- added J5: FlightPin, Connector_PinHeader_2.54mm:PinHeader_1x02_P2.54mm_Horizontal, symbol conn:Conn_01x02
- added R22: 10K, Resistor_SMD:R_0603_1608Metric_Pad1.05x0.95mm_HandSolder, symbol Device:R
Connections:
- net labels added: FlightPin
- wire segments 110 -> 116
Changed lines of the file:
@@
 L Sensor_Motion:LSM303C U?
 U 1 1 5C1D6DCF
-P 6500 4950
+P 7850 4950
 AR Path="/5C13DC71/5C1D6DCF" Ref="U?"  Part="1"
 AR Path="/5C13DC74/5C1D6DCF" Ref="U10"  Part="1"
-F 0 "U10" H 6750 5550 50  0000 C CNN
-F 1 "LSM303C" H 6850 5450 50  0000 C CNN
-F 2 "user:LGA-12_2x2mm_P0.5mm_HandSolder" H 6100 4250 50  0001 L CNN
-F 3 "www.st.com/resource/en/datasheet/lsm303c.pdf" H 6600 4300 50  0001 C CNN
-F 4 "110-6551" H -1300 2100 50  0001 C CNN "品番"
-F 5 "RS" H -1300 2100 50  0001 C CNN "購入先"
-	1    6500 4950
+F 0 "U10" H 8100 5550 50  0000 C CNN
+F 1 "LSM303C" H 8200 5450 50  0000 C CNN
+F 2 "user:LGA-12_2x2mm_P0.5mm_HandSolder" H 7450 4250 50  0001 L CNN
+F 3 "www.st.com/resource/en/datasheet/lsm303c.pdf" H 7950 4300 50  0001 C CNN
+F 4 "110-6551" H 50  2100 50  0001 C CNN "品番"
+F 5 "RS" H 50  2100 50  0001 C CNN "購入先"
+	1    7850 4950
 	1    0    0    -1
 $EndComp
 Wire Wire Line
-	5450 4050 5450 4100
+	6800 4050 6800 4100
 Wire Wire Line
-	5450 4950 5800 4950
+	6800 4950 7150 4950
 Wire Wire Line
-	5800 5050 5450 5050
+	7150 5050 6800 5050
 Wire Wire Line
-	5450 5050 5450 4950
-Connection ~ 5450 4950
+	6800 5050 6800 4950
+Connection ~ 6800 4950
 Wire Wire Line
-	6500 4100 6500 4350
-Connection ~ 5450 4100
+	7850 4100 7850 4350
+Connection ~ 6800 4100
 Wire Wire Line
-	5450 4100 5450 4950
+	6800 4100 6800 4950
 Wire Wire Line
-	6600 4350 6600 4100
+	7950 4350 7950 4100
 Wire Wire Line
-	6600 4100 6500 4100
-Connection ~ 6500 4100
+	7950 4100 7850 4100
+Connection ~ 7850 4100
 $Comp
 L Device:C_Small C?
 U 1 1 5C1D6E08
-P 5450 5450
+P 6800 5450
 AR Path="/5C13DC71/5C1D6E08" Ref="C?"  Part="1"
 AR Path="/5C13DC74/5C1D6E08" Ref="C20"  Part="1"
-F 0 "C20" H 5542 5496 50  0000 L CNN
-F 1 "0.1u" H 5542 5405 50  0000 L CNN
-F 2 "Capacitor_SMD:C_0603_1608Metric_Pad1.05x0.95mm_HandSolder" H 5450 5450 50  0001 C CNN
-F 3 "~" H 5450 5450 50  0001 C CNN
-	1    5450 5450
+F 0 "C20" H 6892 5496 50  0000 L CNN
+F 1 "0.1u" H 6892 5405 50  0000 L CNN
+F 2 "Capacitor_SMD:C_0603_1608Metric_Pad1.05x0.95mm_HandSolder" H 6800 5450 50  0001 C CNN
+F 3 "~" H 6800 5450 50  0001 C CNN
+	1    6800 5450
 	1    0    0    -1
 $EndComp
@@
 L Device:C_Small C?
 U 1 1 5C1D6E0F
-P 7200 5450
+P 8550 5450
 AR Path="/5C13DC71/5C1D6E0F" Ref="C?"  Part="1"
 AR Path="/5C13DC74/5C1D6E0F" Ref="C21"  Part="1"
-F 0 "C21" H 7292 5496 50  0000 L CNN
-F 1 "0.1u" H 7292 5405 50  0000 L CNN
-F 2 "Capacitor_SMD:C_0603_1608Metric_Pad1.05x0.95mm_HandSolder" H 7200 5450 50  0001 C CNN
-F 3 "~" H 7200 5450 50  0001 C CNN
-	1    7200 5450
+F 0 "C21" H 8642 5496 50  0000 L CNN
+F 1 "0.1u" H 8642 5405 50  0000 L CNN
+F 2 "Capacitor_SMD:C_0603_1608Metric_Pad1.05x0.95mm_HandSolder" H 8550 5450 50  0001 C CNN
+F 3 "~" H 8550 5450 50  0001 C CNN
+	1    8550 5450
 	1    0    0    -1
 $EndComp
 Wire Wire Line
-	5450 5350 5450 5050
-Connection ~ 5450 5050
+	6800 5350 6800 5050
+Connection ~ 6800 5050
 Wire Wire Line
-	7200 5350 7200 5150
+	8550 5350 8550 5150
 Wire Wire Line
-	5450 5650 5450 5600
+	6800 5650 6800 5600
 Wire Wire Line
-	5450 5600 6500 5600
+	6800 5600 7850 5600
 Wire Wire Line
-	7200 5600 7200 5550
-Connection ~ 5450 5600
+	8550 5600 8550 5550
+Connection ~ 6800 5600
 Wire Wire Line
-	5450 5600 5450 5550
+	6800 5600 6800 5550
 Wire Wire Line
-	6600 5550 6600 5600
-Connection ~ 6600 5600
+	7950 5550 7950 5600
+Connection ~ 7950 5600
 Wire Wire Line
-	6600 5600 7200 5600
+	7950 5600 8550 5600
 Wire Wire Line
-	6500 5600 6500 5550
-Connection ~ 6500 5600
+	7850 5600 7850 5550
+Connection ~ 7850 5600
 Wire Wire Line
-	6500 5600 6600 5600
+	7850 5600 7950 5600
 $Comp
 L power:VCC #PWR01
 U 1 1 5C1DA52B
-P 5450 4050
-F 0 "#PWR01" H 5450 3900 50  0001 C CNN
-F 1 "VCC" H 5450 4200 50  0000 C CNN
-F 2 "" H 5450 4050 50  0001 C CNN
-F 3 "" H 5450 4050 50  0001 C CNN
-	1    5450 4050
+P 6800 4050
+F 0 "#PWR01" H 6800 3900 50  0001 C CNN
+F 1 "VCC" H 6800 4200 50  0000 C CNN
+F 2 "" H 6800 4050 50  0001 C CNN
+F 3 "" H 6800 4050 50  0001 C CNN
+	1    6800 4050
 	1    0    0    -1
 $EndComp
-Text Label 4900 4850 0    60   ~ 0
+Text Label 6250 4850 0    60   ~ 0
 SDA
-Text Label 4900 4750 0    60   ~ 0
+Text Label 6250 4750 0    60   ~ 0
 SCL
 Wire Wire Line
-	4900 4850 5800 4850
+	6250 4850 7150 4850
 Wire Wire Line
-	4900 4750 5800 4750
+	6250 4750 7150 4750
 Wire Wire Line
-	5450 4100 6500 4100
+	6800 4100 7850 4100
 $Comp
 L EDAMAME_S-rescue:GNDPWR #PWR0160
 U 1 1 5C2B55B9
-P 5450 5650
-F 0 "#PWR0160" H 5450 5450 50  0001 C CNN
-F 1 "GNDPWR" H 5450 5500 50  0000 C CNN
-F 2 "" H 5450 5600 50  0001 C CNN
-F 3 "" H 5450 5600 50  0001 C CNN
-	1    5450 5650
+P 6800 5650
+F 0 "#PWR0160" H 6800 5450 50  0001 C CNN
+F 1 "GNDPWR" H 6800 5500 50  0000 C CNN
+F 2 "" H 6800 5600 50  0001 C CNN
+F 3 "" H 6800 5600 50  0001 C CNN
+	1    6800 5650
 	1    0    0    -1
 $EndComp
+Text Label 2650 1300 2    50   ~ 0
+FlightPin
+Wire Wire Line
+	2050 1300 2650 1300
+$Comp
+L conn:Conn_01x02 J5
+U 1 1 5C211A2B
+P 5100 5200
+F 0 "J5" H 5100 5300 50  0000 C CNN
+F 1 "FlightPin" V 5200 5200 50  0000 C CNN
+F 2 "Connector_PinHeader_2.54mm:PinHeader_1x02_P2.54mm_Horizontal" H 5100 5200 50  0001 C CNN
+F 3 "" H 5100 5200 50  0001 C CNN
+F 4 "" H -2150 1800 50  0001 C CNN "品番"
+F 5 "" H -2150 1800 50  0001 C CNN "購入先"
+	1    5100 5200
+	1    0    0    -1
+$EndComp
+$Comp
+L Device:R R22
+U 1 1 5C21519D
+P 4900 4750
+F 0 "R22" V 4800 4750 50  0000 C CNN
+F 1 "10K" V 4900 4750 50  0000 C CNN
+F 2 "Resistor_SMD:R_0603_1608Metric_Pad1.05x0.95mm_HandSolder" V 4830 4750 50  0001 C CNN
+F 3 "" H 4900 4750 50  0001 C CNN
+	1    4900 4750
+	-1   0    0    1
+$EndComp
+$Comp
+L EDAMAME_S-rescue:GNDPWR #PWR0161
+U 1 1 5C215243
+P 4900 5700
+F 0 "#PWR0161" H 4900 5500 50  0001 C CNN
+F 1 "GNDPWR" H 4900 5550 50  0000 C CNN
+F 2 "" H 4900 5650 50  0001 C CNN
+F 3 "" H 4900 5650 50  0001 C CNN
+	1    4900 5700
+	1    0    0    -1
+$EndComp
+Text Label 4350 5100 0    60   ~ 0
+FlightPin
+$Comp
+L power:VCC #PWR0162
+U 1 1 5C2154E7
+P 4900 4500
+F 0 "#PWR0162" H 4900 4350 50  0001 C CNN
+F 1 "VCC" H 4900 4650 50  0000 C CNN
+F 2 "" H 4900 4500 50  0001 C CNN
+F 3 "" H 4900 4500 50  0001 C CNN
+	1    4900 4500
+	1    0    0    -1
+$EndComp
+Wire Wire Line
+	4900 5200 4900 5100
+Wire Wire Line
+	4900 5300 4900 5700
+Wire Wire Line
+	4350 5100 4900 5100
+Connection ~ 4900 5100
+Wire Wire Line
+	4900 5100 4900 4900
+Wire Wire Line
+	4900 4600 4900 4500
 $EndSCHEMATC
