File: PCB/LED_hachune/LED_hachune.kicad_pcb (KiCad board)
At the start: 2 copper layers, 25 parts, among them J1 POWER, J2 DATA, J3 STlink, U1 M63806KP, U2 TPS63001, U3 STM32F042K6Tx, U4 M63806KP

Commit message: LEDはちゅね 基板製作途中
Parts:
- removed R1, R2, R3, R4, R5, R6: R, Resistor_SMD:R_0603_1608Metric_Pad1.05x0.95mm_HandSolder
- removed U4: M63806KP, Package_SO:SSOP-20_4.4x6.5mm_P0.65mm
- added C5: 1u, Capacitor_SMD:C_0805_2012Metric_Pad1.15x1.40mm_HandSolder, F.Cu at (64.7, 132.6)
- added C6: 0.1u, Capacitor_SMD:C_0603_1608Metric_Pad1.05x0.95mm_HandSolder, F.Cu at (159.5, 155.0)
- added C7: 0.1u, Capacitor_SMD:C_0603_1608Metric_Pad1.05x0.95mm_HandSolder, F.Cu at (162.1, 160.0)
- added D10: S6812Side, user:S6812Side_top, F.Cu at (284.9, 129.2)
- added D11: S6812Side, user:S6812Side_top, F.Cu at (269.6, 138.2)
- added D12: S6812Side, user:S6812Side_top, F.Cu at (280.6, 120.8)
- added D13: S6812Side, user:S6812Side_top, F.Cu at (289.2, 118.0)
- added D14: S6812Side, user:S6812Side_top, F.Cu at (284.9, 118.0)
- added D15: S6812Side, user:S6812Side_top, F.Cu at (278.2, 134.8)
- added D16: S6812Side, user:S6812Side_top, F.Cu at (273.9, 135.4)
- added D17: S6812Side, user:S6812Side_top, F.Cu at (284.9, 126.4)
- added D18: S6812Side, user:S6812Side_top, F.Cu at (305.5, 87.0)
- added D19: S6812Side, user:S6812Side_top, F.Cu at (269.6, 141.0)
- added D20: S6812Side, user:S6812Side_top, F.Cu at (278.2, 132.0)
- added D21: S6812Side, user:S6812Side_top, F.Cu at (273.9, 138.2)
- added D22: S6812Side, user:S6812Side_top, F.Cu at (304.4, 129.6)
- added D23: S6812Side, user:S6812Side_top, F.Cu at (256.8, 138.2)
- added D24: S6812Side, user:S6812Side_top, F.Cu at (305.5, 89.8)
- added D25: S6812Side, user:S6812Side_top, F.Cu at (250.2, 88.7)
- added D26: S6812Side, user:S6812Side_top, F.Cu at (256.5, 82.1)
- added D27: S6812Side, user:S6812Side_top, F.Cu at (258.9, 92.0)
- added D28: S6812Side, user:S6812Side_top, F.Cu at (247.2, 96.3)
- added D29: S6812Side, user:S6812Side_top, F.Cu at (251.4, 67.4)
- added D30: S6812Side, user:S6812Side_top, F.Cu at (281.5, 72.7)
- added D31: S6812Side, user:S6812Side_top, F.Cu at (258.9, 88.7)
- added D32: S6812Side, user:S6812Side_top, F.Cu at (263.1, 88.7)
- added D33: S6812Side, user:S6812Side_top, F.Cu at (275.6, 80.9)
- added D34: S6812Side, user:S6812Side_top, F.Cu at (270.7, 59.7)
- added D35: S6812Side, user:S6812Side_top, F.Cu at (285.2, 66.8)
- added D36: S6812Side, user:S6812Side_top, F.Cu at (276.3, 69.4)
- added D37: S6812Side, user:S6812Side_top, F.Cu at (248.2, 138.2)
- added D38: S6812Side, user:S6812Side_top, F.Cu at (284.9, 123.6)
- added D39: S6812Side, user:S6812Side_top, F.Cu at (248.2, 141.0)
- added D40: S6812Side, user:S6812Side_top, F.Cu at (252.4, 141.0)
- added D41: S6812Side, user:S6812Side_top, F.Cu at (276.3, 123.6)
- added D42: S6812Side, user:S6812Side_top, F.Cu at (256.8, 141.0)
- added D43: S6812Side, user:S6812Side_top, F.Cu at (261.1, 138.2)
- added D44: S6812Side, user:S6812Side_top, F.Cu at (300.1, 129.6)
- added D45: S6812Side, user:S6812Side_top, F.Cu at (280.6, 118.0)
- added D46: S6812Side, user:S6812Side_top, F.Cu at (252.4, 138.2)
- added D47: S6812Side, user:S6812Side_top, F.Cu at (265.4, 135.4)
- added D48: S6812Side, user:S6812Side_top, F.Cu at (265.4, 138.2)
- added D7: S6812Side, user:S6812Side_top, F.Cu at (265.4, 141.0)
- added D8: S6812Side, user:S6812Side_top, F.Cu at (284.9, 120.8)
- added D9: S6812Side, user:S6812Side_top, F.Cu at (308.6, 129.6)
- added J10: LED_T, LED_Frame:LED_socket, F.Cu at (107.6, 85.0)
- added J11: LED_B, LED_Frame:LED_socket, F.Cu at (81.0, 116.6)
- added J12: IN, Connector_JST:JST_EH_S02B-EH_1x02_P2.50mm_Horizontal, F.Cu at (166.5, 168.4)
- added J13: OUT, Connector_JST:JST_EH_S02B-EH_1x02_P2.50mm_Horizontal, F.Cu at (168.5, 156.2)
- added J4: LED_L, LED_Frame:LED_Frame, F.Cu at (262.0, 125.2)
- added J5: LED_L, LED_Frame:LED_socket, F.Cu at (54.4, 85.0)
- added J6: LED_R, LED_Frame:LED_Frame, F.Cu at (262.0, 121.6)
- added J7: LED_T, LED_Frame:LED_Frame, F.Cu at (237.6, 57.8)
- added J8: LED_B, LED_Frame:LED_Frame, F.Cu at (262.0, 117.9)
- added J9: LED_R, LED_Frame:LED_socket, F.Cu at (81.0, 53.4)
- C1: value 100u -> 10u; footprint Capacitor_SMD:C_1210_3225Metric_Pad1.42x2.65mm_HandSolder -> Capacitor_SMD:C_0805_2012Metric_Pad1.15x1.40mm_HandSolder
- D1, D2, D3, D4, D5: value SLC-F11DDA-T1 -> S6812Side; footprint user:SLC-F11DDA-T1 -> user:S6812Side_top
- D6: value LED -> S6812Side; footprint LED_SMD:LED_0603_1608Metric_Pad1.05x0.95mm_HandSolder -> user:S6812Side_top
- U1: value M63806KP -> STM32F042F6Px; footprint Package_SO:SSOP-20_4.4x6.5mm_P0.65mm -> Package_SO:TSSOP-20_4.4x6.5mm_P0.65mm
- U2: value TPS63001 -> XC6202P332PR-G; footprint Package_SON:Texas_S-PVSON-N10_ThermalVias -> Package_TO_SOT_SMD:SOT-89-3
- U3: value STM32F042K6Tx -> TPS63001; footprint Package_QFP:LQFP-32_7x7mm_P0.8mm -> Package_SON:Texas_S-PVSON-N10_ThermalVias; moved to B.Cu
- moved D6 206.3 mm to (280.6, 129.2)
- moved D3 203.9 mm to (276.3, 129.2)
- moved D2 202.9 mm to (280.6, 123.6)
- moved D5 202.2 mm to (280.6, 126.4)
- moved D4 201.4 mm to (269.6, 135.4)
- moved D1 197.8 mm to (261.1, 141.0)
- moved U3 131.2 mm to (152.0, 157.0)
- moved C4 125.3 mm to (152.1, 164.0)
- moved L1 121.8 mm to (146.7, 158.6)
- moved C3 113.7 mm to (151.7, 150.0)
- moved JP1 109.6 mm to (145.7, 152.8)
- moved J3 97.6 mm to (110.1, 136.4), turned to 90 degrees
- moved J2 93.2 mm to (97.5, 136.0)
- moved C1 92.7 mm to (74.7, 132.6), turned to 270 degrees
- moved J1 91.3 mm to (54.5, 136.0)
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Connections:
- C3 pad 1: +BATT -> Net-(C3-Pad1)
- C3 pad 2: GND -> GNDD
- C4 pad 1: +3V3 -> Net-(C4-Pad1)
- C4 pad 2: GND -> GNDD
- D1 pad 1: +3V3 -> Net-(D1-Pad1)
- D2 pad 1: +3V3 -> Net-(D1-Pad3)
- D2 pad 2: Net-(D2-Pad2) -> Net-(D1-Pad2)
- D2 pad 4: Net-(D2-Pad4) -> Net-(D1-Pad4)
- D3 pad 1: +3V3 -> Net-(D2-Pad3)
- D3 pad 2: Net-(D3-Pad2) -> Net-(D1-Pad2)
- D3 pad 4: Net-(D3-Pad4) -> Net-(D1-Pad4)
- D4 pad 1: +3V3 -> Net-(D4-Pad1)
- D4 pad 4: Net-(D4-Pad4) -> Net-(D1-Pad4)
- D5 pad 1: +3V3 -> Net-(D4-Pad3)
- D5 pad 2: Net-(D5-Pad2) -> Net-(D4-Pad2)
- D5 pad 4: Net-(D5-Pad4) -> Net-(D1-Pad4)
- D6 pad 1: Net-(D6-Pad1) -> Net-(D5-Pad3)
- D6 pad 2: Net-(D6-Pad2) -> Net-(D4-Pad2)
- JP1 pad 1: +BATT -> Net-(C3-Pad1)
- U1 pad 1: (no net) -> Net-(U1-Pad1)
- U1 pad 10: GND -> Net-(U1-Pad10)
- U1 pad 11: (no net) -> Net-(U1-Pad11)
- U1 pad 12: Net-(D3-Pad4) -> Net-(U1-Pad12)
- U1 pad 13: Net-(D3-Pad2) -> Net-(U1-Pad13)
- U1 pad 14: Net-(D2-Pad6) -> Net-(U1-Pad14)
- U1 pad 15: Net-(D2-Pad4) -> GND
- U1 pad 16: Net-(D2-Pad2) -> +3V3
- U1 pad 17: Net-(D1-Pad6) -> /TX
- U1 pad 18: Net-(D1-Pad4) -> /RX
- U1 pad 19: Net-(D1-Pad2) -> /SWDIO
- U1 pad 2: /PWM_1R -> /SDA
- U1 pad 20: (no net) -> /SWCLK
- U1 pad 3: /PWM_1G -> /SCL
- U1 pad 4: /PWM_1B -> /NRST
- U1 pad 5: /PWM_2R -> +3V3
- U1 pad 6: /PWM_2G -> /LED_0
- U1 pad 7: /PWM_2B -> /LED_1
- U1 pad 8: /PWM_3R -> /LED_2
- U1 pad 9: /PWM_3G -> /LED_3
- U2 pad 2: Net-(L1-Pad2) -> GND
- U2 pad 3: GND -> +BATT
- U3 pad 1: +3V3 -> Net-(C4-Pad1)
- U3 pad 10: /PWM_LED -> Net-(C4-Pad1)
- U3 pad 11: Net-(U3-Pad11) -> GNDD
- U3 pad 2: /SDA -> Net-(L1-Pad2)
- U3 pad 3: /SCL -> GNDD
- U3 pad 4: /NRST -> Net-(L1-Pad1)
- U3 pad 5: +3V3 -> Net-(C3-Pad1)
- U3 pad 6: /PWM_1R -> Net-(JP1-Pad2)
- U3 pad 7: /PWM_1G -> Net-(C3-Pad1)
- U3 pad 8: /PWM_1B -> Net-(C3-Pad1)
- U3 pad 9: /PWM_2R -> GNDD
Routing:
- net +BATT: track 0.00 -> 267.4 mm
- net /LED_0: track 0.00 -> 223.7 mm, vias 0 -> 8
- net /LED_1: track 0.00 -> 210.8 mm, vias 0 -> 8
- net /LED_2: track 0.00 -> 197.3 mm, vias 0 -> 8
- net /LED_3: track 0.00 -> 190.1 mm, vias 0 -> 7
- net GND: track 0.00 -> 53.2 mm, vias 0 -> 8
- net /SWDIO: track 0.00 -> 29.4 mm
- net /TX: track 0.00 -> 27.9 mm
- net /RX: track 0.00 -> 27.5 mm
- net /SWCLK: track 0.00 -> 26.2 mm
- net +3V3: track 0.00 -> 19.9 mm
- net /SDA: track 0.00 -> 16.3 mm
- net /SCL: track 0.00 -> 14.4 mm
- added copper zone on B.Cu, net GND
- added copper zone on F.Cu, net GND
Other:
- board outline added: 180 x 100 mm
- net class Default: clearance 0.2 -> 0.2032; trace_width 0.25 -> 0.2032; via_dia 0.8 -> 0.2032; via_drill 0.4 -> 0.1524
- rule pad_to_mask_clearance: 0.2 -> 0
- rule trace_clearance: 0.2 -> 0.2032
- rule trace_min: 0.2 -> 0.1524
- rule via_min_drill: 0.3 -> 0.1524
- rule via_min_size: 0.4 -> 0.1524
