File: PCB/LED_hachune/LED_hachune.sch (KiCad schematic (older format))
At the start: 25 parts, among them J1 POWER, J2 DATA, J3 Debug, U1 M63806KP, U2 TPS63000, U3 STM32F042K6Tx, U4 M63806KP

Commit message: 回路変更(フットプリントの割り当てはまだ）
Parts:
- U2: value TPS63000 -> TPS63001
Changed lines of the file:
@@
 EESchema Schematic File Version 4
+LIBS:LED_hachune-cache
 EELAYER 26 0
 EELAYER END
@@
 F 3 "~" H 6750 1750 50  0001 C CNN
 	1    6750 1800
-	0    1    -1   0
+	0    -1   -1   0
 $EndComp
 $Comp
@@
 F 3 "~" H 7650 1750 50  0001 C CNN
 	1    7650 1800
-	0    1    -1   0
+	0    -1   -1   0
 $EndComp
 $Comp
@@
 F 3 "~" H 8550 1750 50  0001 C CNN
 	1    8550 1800
-	0    1    -1   0
+	0    -1   -1   0
 $EndComp
 $Comp
@@
 F 3 "~" H 9450 1750 50  0001 C CNN
 	1    9450 1800
-	0    1    -1   0
+	0    -1   -1   0
 $EndComp
 Text Label 2750 3600 0    50   ~ 0
@@
 F 3 "~" H 10350 1750 50  0001 C CNN
 	1    10350 1800
-	0    1    -1   0
+	0    -1   -1   0
 $EndComp
 $Comp
@@
 L Device:LED D6
 U 1 1 5BE5C741
-P 10850 1800
-F 0 "D6" V 10888 1683 50  0000 R CNN
-F 1 "LED" V 10797 1683 50  0000 R CNN
-F 2 "" H 10850 1800 50  0001 C CNN
-F 3 "~" H 10850 1800 50  0001 C CNN
-	1    10850 1800
+P 10950 1800
+F 0 "D6" V 10988 1683 50  0000 R CNN
+F 1 "LED" V 10897 1683 50  0000 R CNN
+F 2 "" H 10950 1800 50  0001 C CNN
+F 3 "~" H 10950 1800 50  0001 C CNN
+	1    10950 1800
 	0    -1   -1   0
 $EndComp
 Wire Wire Line
-	10850 1950 10850 4150
-Wire Wire Line
-	10850 4150 6250 4150
+	10950 1950 10950 4150
 Text Label 4550 2600 2    50   ~ 0
 PWM_LED
@@
 L Device:R R1
 U 1 1 5BE63394
-P 6950 1350
-F 0 "R1" H 7020 1396 50  0000 L CNN
-F 1 "R" H 7020 1305 50  0000 L CNN
-F 2 "" V 6880 1350 50  0001 C CNN
-F 3 "~" H 6950 1350 50  0001 C CNN
-	1    6950 1350
-	1    0    0    -1
+P 6550 1350
+F 0 "R1" H 6620 1396 50  0000 L CNN
+F 1 "R" H 6620 1305 50  0000 L CNN
+F 2 "" V 6480 1350 50  0001 C CNN
+F 3 "~" H 6550 1350 50  0001 C CNN
+	1    6550 1350
+	-1   0    0    -1
 $EndComp
 $Comp
@@
 F 3 "" H 6750 1100 50  0001 C CNN
 	1    6750 1100
-	1    0    0    -1
-$EndComp
-Wire Wire Line
-	6950 1200 6950 1150
-Wire Wire Line
-	6950 1150 6750 1150
+	-1   0    0    -1
+$EndComp
+Wire Wire Line
+	6550 1200 6550 1150
+Wire Wire Line
+	6550 1150 6750 1150
 Wire Wire Line
 	6750 1150 6750 1100
 Wire Wire Line
-	6750 1150 6550 1150
-Wire Wire Line
-	6550 1150 6550 1600
+	6750 1150 6950 1150
+Wire Wire Line
+	6950 1150 6950 1600
 Connection ~ 6750 1150
 Wire Wire Line
 	6750 1600 6750 1150
 Wire Wire Line
-	6950 1500 6950 1600
+	6550 1500 6550 1600
 $Comp
 L Device:R R2
 U 1 1 5BE720A1
-P 7850 1350
-F 0 "R2" H 7920 1396 50  0000 L CNN
-F 1 "R" H 7920 1305 50  0000 L CNN
-F 2 "" V 7780 1350 50  0001 C CNN
-F 3 "~" H 7850 1350 50  0001 C CNN
-	1    7850 1350
-	1    0    0    -1
+P 7450 1350
+F 0 "R2" H 7520 1396 50  0000 L CNN
+F 1 "R" H 7520 1305 50  0000 L CNN
+F 2 "" V 7380 1350 50  0001 C CNN
+F 3 "~" H 7450 1350 50  0001 C CNN
+	1    7450 1350
+	-1   0    0    -1
 $EndComp
 $Comp
@@
 F 3 "" H 7650 1100 50  0001 C CNN
 	1    7650 1100
-	1    0    0    -1
-$EndComp
-Wire Wire Line
-	7850 1200 7850 1150
-Wire Wire Line
-	7850 1150 7650 1150
+	-1   0    0    -1
+$EndComp
+Wire Wire Line
+	7450 1200 7450 1150
+Wire Wire Line
+	7450 1150 7650 1150
 Wire Wire Line
 	7650 1150 7650 1100
 Wire Wire Line
-	7650 1150 7450 1150
-Wire Wire Line
-	7450 1150 7450 1600
+	7650 1150 7850 1150
+Wire Wire Line
+	7850 1150 7850 1600
 Connection ~ 7650 1150
 Wire Wire Line
 	7650 1600 7650 1150
 Wire Wire Line
-	7850 1500 7850 1600
+	7450 1500 7450 1600
 $Comp
 L Device:R R3
 U 1 1 5BE77FD8
-P 8750 1350
-F 0 "R3" H 8820 1396 50  0000 L CNN
-F 1 "R" H 8820 1305 50  0000 L CNN
-F 2 "" V 8680 1350 50  0001 C CNN
-F 3 "~" H 8750 1350 50  0001 C CNN
-	1    8750 1350
-	1    0    0    -1
+P 8350 1350
+F 0 "R3" H 8420 1396 50  0000 L CNN
+F 1 "R" H 8420 1305 50  0000 L CNN
+F 2 "" V 8280 1350 50  0001 C CNN
+F 3 "~" H 8350 1350 50  0001 C CNN
+	1    8350 1350
+	-1   0    0    -1
 $EndComp
 $Comp
@@
 F 3 "" H 8550 1100 50  0001 C CNN
 	1    8550 1100
-	1    0    0    -1
-$EndComp
-Wire Wire Line
-	8750 1200 8750 1150
-Wire Wire Line
-	8750 1150 8550 1150
+	-1   0    0    -1
+$EndComp
+Wire Wire Line
+	8350 1200 8350 1150
+Wire Wire Line
+	8350 1150 8550 1150
 Wire Wire Line
 	8550 1150 8550 1100
 Wire Wire Line
-	8550 1150 8350 1150
-Wire Wire Line
-	8350 1150 8350 1600
+	8550 1150 8750 1150
+Wire Wire Line
+	8750 1150 8750 1600
 Connection ~ 8550 1150
 Wire Wire Line
 	8550 1600 8550 1150
 Wire Wire Line
-	8750 1500 8750 1600
+	8350 1500 8350 1600
 $Comp
 L Device:R R4
 U 1 1 5BE7B1BB
-P 9650 1350
-F 0 "R4" H 9720 1396 50  0000 L CNN
-F 1 "R" H 9720 1305 50  0000 L CNN
-F 2 "" V 9580 1350 50  0001 C CNN
-F 3 "~" H 9650 1350 50  0001 C CNN
-	1    9650 1350
-	1    0    0    -1
+P 9250 1350
+F 0 "R4" H 9320 1396 50  0000 L CNN
+F 1 "R" H 9320 1305 50  0000 L CNN
+F 2 "" V 9180 1350 50  0001 C CNN
+F 3 "~" H 9250 1350 50  0001 C CNN
+	1    9250 1350
+	-1   0    0    -1
 $EndComp
 $Comp
@@
 F 3 "" H 9450 1100 50  0001 C CNN
 	1    9450 1100
-	1    0    0    -1
-$EndComp
-Wire Wire Line
-	9650 1200 9650 1150
-Wire Wire Line
-	9650 1150 9450 1150
+	-1   0    0    -1
+$EndComp
+Wire Wire Line
+	9250 1200 9250 1150
+Wire Wire Line
+	9250 1150 9450 1150
 Wire Wire Line
 	9450 1150 9450 1100
 Wire Wire Line
-	9450 1150 9250 1150
-Wire Wire Line
-	9250 1150 9250 1600
+	9450 1150 9650 1150
+Wire Wire Line
+	9650 1150 9650 1600
 Connection ~ 9450 1150
 Wire Wire Line
 	9450 1600 9450 1150
 Wire Wire Line
-	9650 1500 9650 1600
+	9250 1500 9250 1600
 $Comp
 L Device:R R5
 U 1 1 5BE7E857
-P 10550 1350
-F 0 "R5" H 10620 1396 50  0000 L CNN
-F 1 "R" H 10620 1305 50  0000 L CNN
-F 2 "" V 10480 1350 50  0001 C CNN
-F 3 "~" H 10550 1350 50  0001 C CNN
-	1    10550 1350
-	1    0    0    -1
+P 10150 1350
+F 0 "R5" H 10220 1396 50  0000 L CNN
+F 1 "R" H 10220 1305 50  0000 L CNN
+F 2 "" V 10080 1350 50  0001 C CNN
+F 3 "~" H 10150 1350 50  0001 C CNN
+	1    10150 1350
+	-1   0    0    -1
 $EndComp
 $Comp
@@
 F 3 "" H 10350 1100 50  0001 C CNN
 	1    10350 1100
-	1    0    0    -1
-$EndComp
-Wire Wire Line
-	10550 1200 10550 1150
-Wire Wire Line
-	10550 1150 10350 1150
+	-1   0    0    -1
+$EndComp
+Wire Wire Line
+	10150 1200 10150 1150
+Wire Wire Line
+	10150 1150 10350 1150
 Wire Wire Line
 	10350 1150 10350 1100
 Wire Wire Line
-	10350 1150 10150 1150
-Wire Wire Line
-	10150 1150 10150 1600
+	10350 1150 10550 1150
+Wire Wire Line
+	10550 1150 10550 1600
 Connection ~ 10350 1150
 Wire Wire Line
 	10350 1600 10350 1150
 Wire Wire Line
-	10550 1500 10550 1600
+	10150 1500 10150 1600
 $Comp
 L Device:R R6
 U 1 1 5BE823BE
-P 10850 1350
-F 0 "R6" H 10920 1396 50  0000 L CNN
-F 1 "R" H 10920 1305 50  0000 L CNN
-F 2 "" V 10780 1350 50  0001 C CNN
-F 3 "~" H 10850 1350 50  0001 C CNN
-	1    10850 1350
+P 10950 1350
+F 0 "R6" H 11020 1396 50  0000 L CNN
+F 1 "R" H 11020 1305 50  0000 L CNN
+F 2 "" V 10880 1350 50  0001 C CNN
+F 3 "~" H 10950 1350 50  0001 C CNN
+	1    10950 1350
 	1    0    0    -1
 $EndComp
@@
 L power:+3.3V #PWR012
 U 1 1 5BE823C5
-P 10850 1150
-F 0 "#PWR012" H 10850 1000 50  0001 C CNN
-F 1 "+3.3V" H 10865 1323 50  0000 C CNN
-F 2 "" H 10850 1150 50  0001 C CNN
-F 3 "" H 10850 1150 50  0001 C CNN
-	1    10850 1150
-	1    0    0    -1
-$EndComp
-Wire Wire Line
-	10850 1200 10850 1150
+P 10950 1150
+F 0 "#PWR012" H 10950 1000 50  0001 C CNN
+F 1 "+3.3V" H 10965 1323 50  0000 C CNN
+F 2 "" H 10950 1150 50  0001 C CNN
+F 3 "" H 10950 1150 50  0001 C CNN
+	1    10950 1150
+	1    0    0    -1
+$EndComp
+Wire Wire Line
+	10950 1200 10950 1150
 Wire Wire Line
 	5000 2900 5450 2900
@@
 P 1750 2750
 F 0 "U2" H 1750 3417 50  0000 C CNN
-F 1 "TPS63000" H 1750 3326 50  0000 C CNN
+F 1 "TPS63001" H 1750 3326 50  0000 C CNN
 F 2 "Package_SON:Texas_S-PWSON-N10_ThermalVias" H 1750 2100 50  0001 C CNN
 F 3 "https://strawberry-linux.com/pub/tps63000.pdf" H 1750 2750 50  0001 C CNN
@@
 	3650 1050 3650 950
 Wire Wire Line
-	10850 1500 10850 1650
+	10950 1500 10950 1650
+Wire Wire Line
+	6250 4150 10950 4150
 $EndSCHEMATC

Commit message: フットプリント割当
Parts:
- removed J3: Debug, symbol Connector_Generic:Conn_01x06
- added J3: STlink, user:STlink, symbol Connector_Generic:Conn_01x05
- C1: footprint (none) -> Capacitor_SMD:C_1210_3225Metric_Pad1.42x2.65mm_HandSolder
- C2: footprint (none) -> Capacitor_SMD:C_0603_1608Metric_Pad1.05x0.95mm_HandSolder
- C3, C4: footprint (none) -> Capacitor_SMD:C_0805_2012Metric_Pad1.15x1.40mm_HandSolder
- D1, D2, D3, D4, D5: footprint (none) -> user:SLC-F11DDA-T1; symbol Device:LED_RGB -> user_library:SLC-F11DDA-T1
- D6: footprint (none) -> LED_SMD:LED_0603_1608Metric_Pad1.05x0.95mm_HandSolder
- J1: footprint (none) -> Connector_JST:JST_EH_S02B-EH_1x02_P2.50mm_Horizontal
- J2: footprint (none) -> Connector_JST:JST_EH_S03B-EH_1x03_P2.50mm_Horizontal
- JP1: footprint (none) -> Jumper:SolderJumper-2_P1.3mm_Open_Pad1.0x1.5mm
- L1: footprint (none) -> user:inductor_VLF4012-2R2
- R1, R2, R3, R4, R5, R6: footprint (none) -> Resistor_SMD:R_0603_1608Metric_Pad1.05x0.95mm_HandSolder
- U1, U4: footprint (none) -> Package_SO:SSOP-20_4.4x6.5mm_P0.65mm
- U2: footprint Package_SON:Texas_S-PWSON-N10_ThermalVias -> Package_SON:Texas_S-PVSON-N10_ThermalVias
Connections:
- wire segments 165 -> 164

Commit message: LEDはちゅね 基板製作途中
Parts:
- removed D1, D2, D3, D4, D5: SLC-F11DDA-T1, user:SLC-F11DDA-T1, symbol user_library:SLC-F11DDA-T1
- removed D6: LED, LED_SMD:LED_0603_1608Metric_Pad1.05x0.95mm_HandSolder, symbol Device:LED
- removed R1, R2, R3, R4, R5, R6: R, Resistor_SMD:R_0603_1608Metric_Pad1.05x0.95mm_HandSolder, symbol Device:R
- removed U1, U4: M63806KP, Package_SO:SSOP-20_4.4x6.5mm_P0.65mm, symbol user_library:M63806P
- removed U3: STM32F042K6Tx, Package_QFP:LQFP-32_7x7mm_P0.8mm, symbol MCU_ST_STM32F0:STM32F042K6Tx
- added C5: 1u, Capacitor_SMD:C_0805_2012Metric_Pad1.15x1.40mm_HandSolder, symbol Device:C
- added C6, C7: 0.1u, Capacitor_SMD:C_0603_1608Metric_Pad1.05x0.95mm_HandSolder, symbol Device:C
- added D1, D10, D11, D12, D13, D14, D15, D16, D17, D18, D19, D2, D20, D21, D22, D23, D24, D3, D4, D5, D6, D7, D8, D9: S6812Side, user:S6812Side_top, symbol user_library:S6812Side
- added J10: LED_T, LED_Frame:LED_socket, symbol Connector:Conn_01x14_Female
- added J11: LED_B, LED_Frame:LED_socket, symbol Connector:Conn_01x14_Female
- added J12: IN, Connector_JST:JST_EH_S02B-EH_1x02_P2.50mm_Horizontal, symbol Connector_Generic:Conn_01x02
- added J13: OUT, Connector_JST:JST_EH_S02B-EH_1x02_P2.50mm_Horizontal, symbol Connector_Generic:Conn_01x02
- added J4, J6: LED_L, LED_Frame:LED_Frame, symbol Connector:Conn_01x14_Male
- added J5: LED_L, LED_Frame:LED_socket, symbol Connector:Conn_01x14_Female
- added J9: LED_R, LED_Frame:LED_socket, symbol Connector:Conn_01x14_Female
- added U1: STM32F042F6Px, Package_SO:TSSOP-20_4.4x6.5mm_P0.65mm, symbol MCU_ST_STM32F0:STM32F042F6Px
- added U2: XC6202P332PR-G, Package_TO_SOT_SMD:SOT-89-3, symbol Regulator_Linear:L78L18_SOT89
- C1: value 100u -> 10u; footprint Capacitor_SMD:C_1210_3225Metric_Pad1.42x2.65mm_HandSolder -> Capacitor_SMD:C_0805_2012Metric_Pad1.15x1.40mm_HandSolder
- renumbered U2 to U3
Connections:
- net labels added: GNDD, LED_0, LED_1, LED_2, LED_3
- net labels removed: PWM_1B, PWM_1G, PWM_1R, PWM_2B, PWM_2G, PWM_2R, PWM_3B, PWM_3G, PWM_3R, PWM_4B, PWM_4G, PWM_4R, PWM_LED, Rx, Tx
- wire segments 164 -> 302
- no-connect marks 2 -> 1
Other:
- note added: "3.3V\n150mA"

Commit message: LED_hacune レビュー1
Parts:
- added D25, D26, D27, D28, D29, D30, D31, D32, D33, D34, D35, D36, D37, D38, D39, D40, D41, D42, D43, D44, D45, D46, D47, D48: S6812Side, user:S6812Side_top, symbol user_library:S6812Side
- added J7, J8: LED_L, LED_Frame:LED_Frame, symbol Connector:Conn_01x14_Male
Connections:
- wire segments 302 -> 460
