File: PCB/LED_hachune/LED_hachune_2.kicad_pcb (KiCad board)
At the start: 2 copper layers, 70 x 100 mm, 35 parts, among them J12 IN, J13 OUT, J4 LED_L, J6 LED_L, U3 TPS63001

Commit message: LED_hacune レビュー1
Parts:
- added D25: S6812Side, user:S6812Side_top, F.Cu at (88.5, 127.5)
- added D26: S6812Side, user:S6812Side_top, F.Cu at (88.5, 109.5)
- added D27: S6812Side, user:S6812Side_top, F.Cu at (88.5, 92.0)
- added D28: S6812Side, user:S6812Side_top, F.Cu at (91.0, 132.0)
- added D29: S6812Side, user:S6812Side_top, F.Cu at (91.0, 114.5)
- added D30: S6812Side, user:S6812Side_top, F.Cu at (91.0, 97.0)
- added D31: S6812Side, user:S6812Side_top, F.Cu at (93.5, 127.5)
- added D32: S6812Side, user:S6812Side_top, F.Cu at (93.5, 109.5)
- added D33: S6812Side, user:S6812Side_top, F.Cu at (93.5, 92.0)
- added D34: S6812Side, user:S6812Side_top, F.Cu at (96.0, 132.0)
- added D35: S6812Side, user:S6812Side_top, F.Cu at (96.0, 114.5)
- added D36: S6812Side, user:S6812Side_top, F.Cu at (96.0, 97.0)
- added D37: S6812Side, user:S6812Side_top, F.Cu at (102.5, 127.5)
- added D38: S6812Side, user:S6812Side_top, F.Cu at (102.5, 109.5)
- added D39: S6812Side, user:S6812Side_top, F.Cu at (102.5, 92.0)
- added D40: S6812Side, user:S6812Side_top, F.Cu at (105.0, 132.0)
- added D41: S6812Side, user:S6812Side_top, F.Cu at (105.0, 114.5)
- added D42: S6812Side, user:S6812Side_top, F.Cu at (105.0, 97.0)
- added D43: S6812Side, user:S6812Side_top, F.Cu at (107.5, 127.5)
- added D44: S6812Side, user:S6812Side_top, F.Cu at (107.5, 109.5)
- added D45: S6812Side, user:S6812Side_top, F.Cu at (107.5, 92.0)
- added D46: S6812Side, user:S6812Side_top, F.Cu at (110.0, 132.0)
- added D47: S6812Side, user:S6812Side_top, F.Cu at (110.0, 114.5)
- added D48: S6812Side, user:S6812Side_top, F.Cu at (110.0, 97.0)
- added J7: LED_L, LED_Frame:LED_Frame, B.Cu at (86.5, 110.0)
- added J8: LED_L, LED_Frame:LED_Frame, B.Cu at (100.5, 110.0)
Routing:
- net Net-(D37-Pad4): track 0.00 -> 110.6 mm, vias 0 -> 14
- net Net-(D25-Pad4): track 0.00 -> 110.6 mm, vias 0 -> 14
- net Net-(D37-Pad2): track 0.00 -> 100.9 mm, vias 0 -> 5
- net Net-(D25-Pad2): track 0.00 -> 100.9 mm, vias 0 -> 5
- net Net-(D46-Pad1): track 0.00 -> 25.0 mm, vias 0 -> 1
- net Net-(D34-Pad1): track 0.00 -> 25.0 mm, vias 0 -> 1
- net Net-(D40-Pad1): track 0.00 -> 19.0 mm, vias 0 -> 1
- net Net-(D28-Pad1): track 0.00 -> 19.0 mm, vias 0 -> 1
- net Net-(D38-Pad3): track 0.00 -> 18.3 mm
- net Net-(D26-Pad3): track 0.00 -> 18.3 mm
- net Net-(D43-Pad1): track 0.00 -> 17.5 mm, vias 0 -> 1
- net Net-(D31-Pad1): track 0.00 -> 17.5 mm, vias 0 -> 1
- net Net-(D44-Pad3): track 0.00 -> 17.2 mm, vias 0 -> 2
- net Net-(D32-Pad3): track 0.00 -> 17.2 mm, vias 0 -> 2
- net Net-(D40-Pad3): track 0.00 -> 17.2 mm, vias 0 -> 2
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- added copper zone on B.Cu, net Net-(D25-Pad4)
- added copper zone on F.Cu, net Net-(D25-Pad4)
- added copper zone on B.Cu, net Net-(D37-Pad4)
- added copper zone on F.Cu, net Net-(D37-Pad4)

Commit message: LED_hachune PCB NT加賀
Parts:
- moved C3 29.0 mm to (73.5, 58.8)
- moved C4 29.0 mm to (65.5, 58.5)
- moved C6 29.0 mm to (75.5, 58.8)
- moved C7 29.0 mm to (63.5, 58.5)
- moved J12 29.0 mm to (78.0, 57.5)
- moved J13 29.0 mm to (61.0, 59.8)
- moved JP1 29.0 mm to (74.4, 52.5)
- moved L1 29.0 mm to (69.8, 62.5)
- moved U3 29.0 mm to (69.8, 56.5)
Other:
- outline, holes or cut-outs redrawn
- board text added: "2018/11/23 @n_yosihisa"
- board text added: "IN"
- board text added: "OUT"
