File: PCB/EDAMAME_S_M_PowerBoard/EDAMAME_S_M_PowerBoard.kicad_pcb (KiCad board)
At the start: 2 copper layers, 180 x 100 mm, 73 parts, among them J1 POWER, J10 LED_T, J11 LED_B, J12 IN, J13 OUT, J2 DATA, J3 STlink, J4 LED_L, J5 LED_L, J6 LED_R, J7 LED_T, J8 LED_B, J9 LED_R, U1 STM32F042F6Px, U2 XC6202P332PR-G, U3 TPS63001

Commit message: Add PCB layout
Parts:
- removed C3, C4: 10u, Capacitor_SMD:C_0805_2012Metric_Pad1.15x1.40mm_HandSolder
- removed C5: 1u, Capacitor_SMD:C_0805_2012Metric_Pad1.15x1.40mm_HandSolder
- removed C6, C7: 0.1u, Capacitor_SMD:C_0603_1608Metric_Pad1.05x0.95mm_HandSolder
- removed D10, D11, D12, D13, D14, D15, D16, D17, D18, D19, D2, D20, D21, D22, D23, D24, D25, D26, D27, D28, D29, D3, D30, D31, D32, D33, D34, D35, D36, D37, D38, D39, D4, D40, D41, D42, D43, D44, D45, D46, D47, D48, D5, D6, D7, D8, D9: S6812Side, user:S6812Side_top
- removed J10: LED_T, LED_Frame:LED_socket
- removed J11: LED_B, LED_Frame:LED_socket
- removed J12: IN, Connector_JST:JST_EH_S02B-EH_1x02_P2.50mm_Horizontal
- removed J13: OUT, Connector_JST:JST_EH_S02B-EH_1x02_P2.50mm_Horizontal
- removed J8: LED_B, LED_Frame:LED_Frame
- removed J9: LED_R, LED_Frame:LED_socket
- removed JP1: EN, Jumper:SolderJumper-2_P1.3mm_Open_Pad1.0x1.5mm
- removed U2: XC6202P332PR-G, Package_TO_SOT_SMD:SOT-89-3
- removed U3: TPS63001, Package_SON:Texas_S-PVSON-N10_ThermalVias
- added BT1: Li-Po, Connector_JST:JST_EH_S02B-EH_1x02_P2.50mm_Horizontal, B.Cu at (58.5, 132.0)
- added G***: LOGO, logo:SOMESAT_edamame_s_logo, B.Cu at (93.8, 58.5)
- added R1: R, Resistor_SMD:R_0603_1608Metric_Pad1.05x0.95mm_HandSolder, F.Cu at (105.3, 104.1)
- added R2: R, Resistor_SMD:R_0603_1608Metric_Pad1.05x0.95mm_HandSolder, F.Cu at (55.1, 67.3)
- added SW1: power, user:SS-12D01-VG4, F.Cu at (105.0, 111.8)
- C2: value 0.1u -> 10u; footprint Capacitor_SMD:C_0603_1608Metric_Pad1.05x0.95mm_HandSolder -> Capacitor_SMD:C_0805_2012Metric_Pad1.15x1.40mm_HandSolder
- D1: value S6812Side -> LED_Small; footprint user:S6812Side_top -> LED_SMD:LED_0603_1608Metric_Pad1.05x0.95mm_HandSolder
- J1: value POWER -> Charge
- J2: value DATA -> IMU_Power; footprint Connector_JST:JST_EH_S03B-EH_1x03_P2.50mm_Horizontal -> Connector_JST:JST_EH_B02B-EH-A_1x02_P2.50mm_Vertical; moved to B.Cu
- J3: value STlink -> IMU_Debug; moved to B.Cu
- J4: value LED_L -> flight_pin; footprint LED_Frame:LED_Frame -> Connector_JST:JST_EH_S02B-EH_1x02_P2.50mm_Horizontal; moved to B.Cu
- J5: value LED_L -> IMU_Board; footprint LED_Frame:LED_socket -> Connector_PinHeader_1.27mm:PinHeader_2x05_P1.27mm_Vertical; moved to B.Cu
- J6: value LED_R -> OBC_Board; footprint LED_Frame:LED_Frame -> Connector_PinSocket_2.54mm:PinSocket_2x19_P2.54mm_Vertical; moved to B.Cu
- J7: value LED_T -> LED_Board; footprint LED_Frame:LED_Frame -> Connector_JST:JST_EH_S04B-EH_1x04_P2.50mm_Horizontal
- L1: value 2.2uH VLF4012-2R2 -> 2.2uH
- U1: value STM32F042F6Px -> TPS63002; footprint Package_SO:TSSOP-20_4.4x6.5mm_P0.65mm -> Package_SON:Texas_S-PVSON-N10_ThermalVias
- moved J6 211.9 mm to (58.8, 61.3), turned to 180 degrees
- moved J4 198.0 mm to (79.9, 47.5), turned to 180 degrees
- moved D1 161.1 mm to (105.3, 99.9), turned to 270 degrees
- moved J7 150.5 mm to (104.5, 128.0), turned to 90 degrees
- moved J3 89.2 mm to (73.5, 55.0), turned to 180 degrees
- moved L1 72.2 mm to (79.2, 133.1), turned to 180 degrees
- moved J2 33.0 mm to (64.9, 131.0), turned to 90 degrees
- moved J5 27.5 mm to (68.0, 61.1), turned to 270 degrees
- moved J1 19.2 mm to (61.7, 118.2), turned to 90 degrees
- moved C1 10.2 mm to (83.6, 127.7)
- moved U1 7.08 mm to (79.2, 128.1), turned to 90 degrees
- moved C2 6.68 mm to (75.0, 127.7)
Connections:
- C1 pad 1: +3V3 -> +BATT
- C2 pad 1: +3V3 -> +5V
- D1 pad 1: Net-(D1-Pad1) -> GND
- J1 pad 1: +BATT -> Net-(BT1-Pad1)
- J2 pad 1: /SCL -> GND
- J2 pad 2: /SDA -> +5V
- J3 pad 1: /TX -> /IMU_TX
- J3 pad 2: /RX -> /IMU_RX
- J4 pad 1: Net-(D1-Pad4) -> /flight_pin
- J4 pad 2: Net-(D1-Pad4) -> GND
- J5 pad 1: GND -> /SWDIO
- J5 pad 10: /LED_1 -> (no net)
- J5 pad 3: +BATT -> /SWCLK
- J5 pad 4: /LED_0 -> /IMU_TX
- J5 pad 5: /LED_1 -> /NRST
- J5 pad 6: /LED_2 -> /IMU_RX
- J5 pad 7: /LED_3 -> (no net)
- J5 pad 8: /LED_3 -> (no net)
- J5 pad 9: /LED_2 -> (no net)
- J6 pad 1: Net-(D13-Pad4) -> +5V
- J6 pad 10: Net-(D16-Pad1) -> Net-(J6-Pad10)
- J6 pad 11: Net-(D13-Pad1) -> Net-(J6-Pad11)
- J6 pad 12: Net-(D13-Pad2) -> Net-(J6-Pad12)
- J6 pad 13: Net-(D13-Pad4) -> Net-(J6-Pad13)
- J6 pad 14: Net-(D13-Pad4) -> Net-(J6-Pad14)
- J6 pad 2: Net-(D13-Pad4) -> +5V
- J6 pad 3: Net-(D13-Pad2) -> +5V
- J6 pad 4: Net-(D13-Pad1) -> +5V
- J6 pad 5: Net-(D16-Pad1) -> +3V3
- J6 pad 6: Net-(D19-Pad1) -> Net-(J6-Pad6)
- J6 pad 7: Net-(D22-Pad1) -> GND
- J6 pad 8: Net-(D22-Pad1) -> GND
- J6 pad 9: Net-(D19-Pad1) -> /flight_pin
- J7 pad 1: Net-(D25-Pad4) -> /SCL
- J7 pad 2: Net-(D25-Pad4) -> /SDA
- J7 pad 3: Net-(D25-Pad2) -> +5V
- J7 pad 4: Net-(D25-Pad1) -> GND
- U1 pad 1: Net-(U1-Pad1) -> +5V
- U1 pad 10: Net-(U1-Pad10) -> +5V
- U1 pad 11: Net-(U1-Pad11) -> GND
- U1 pad 2: /SDA -> Net-(L1-Pad2)
- U1 pad 3: /SCL -> GND
- U1 pad 4: /NRST -> Net-(L1-Pad1)
- U1 pad 5: +3V3 -> +BATT
- U1 pad 6: /LED_0 -> +BATT
- U1 pad 7: /LED_1 -> +BATT
- U1 pad 8: /LED_2 -> +BATT
- U1 pad 9: /LED_3 -> GND
Routing:
- net /LED_0: track 223.7 -> 0.00 mm, vias 8 -> 0
- net +BATT: track 267.4 -> 49.0 mm
- net /LED_1: track 210.8 -> 0.00 mm, vias 8 -> 0
- net +5V: track 0.00 -> 197.8 mm
- net /LED_2: track 197.3 -> 0.00 mm, vias 8 -> 0
- net /LED_3: track 190.1 -> 0.00 mm, vias 7 -> 0
- net /SCL: track 14.4 -> 91.7 mm
- net /SDA: track 16.3 -> 88.8 mm
- net Net-(BT1-Pad1): track 0.00 -> 60.3 mm
- net /flight_pin: track 0.00 -> 51.8 mm
- net /IMU_RX: track 0.00 -> 43.6 mm
- net /IMU_TX: track 0.00 -> 41.6 mm
- net /TX: track 27.9 -> 0.00 mm
- net /RX: track 27.5 -> 0.00 mm
- net /SWDIO: track 29.4 -> 6.54 mm
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Other:
- board size 180 x 100 mm -> 58 x 100 mm
- board text added: "+ -"
- board text added: "OFF ON"
- board text added: "SOMESAT EDAMAME S Mission PowerBoard V1.0 @n_yosihisa 2019/01/20"
