File: PCB/EDAMAME_S_M_PowerBoard/EDAMAME_S_M_PowerBoard.sch (KiCad schematic (older format))
At the start: 16 parts, among them J1 Charge, J2 IMU_Power, J3 IMU_Debug, J4 flight_pin, J5 IMU_Board, J6 OBC_Board, J7 LED_Board, SW1 power, U1 TPS63002

Commit message: Add PCB layout
Parts:
- BT1: value Li-Po 3.7V 800mAh -> Li-Po; footprint Connector_JST:JST_XH_S02B-XH-A-1_1x02_P2.50mm_Horizontal -> Connector_JST:JST_EH_S02B-EH_1x02_P2.50mm_Horizontal
- J1: footprint Connector_JST:JST_XH_S02B-XH-A_1x02_P2.50mm_Horizontal -> Connector_JST:JST_EH_S02B-EH_1x02_P2.50mm_Horizontal
- J2: footprint Connector_JST:JST_XH_S02B-XH-A_1x02_P2.50mm_Horizontal -> Connector_JST:JST_EH_B02B-EH-A_1x02_P2.50mm_Vertical
- J4: footprint Connector_JST:JST_XH_S02B-XH-A-1_1x02_P2.50mm_Horizontal -> Connector_JST:JST_EH_S02B-EH_1x02_P2.50mm_Horizontal
- J7: footprint Connector_JST:JST_XH_S04B-XH-A_1x04_P2.50mm_Horizontal -> Connector_JST:JST_EH_S04B-EH_1x04_P2.50mm_Horizontal
- U1: footprint Package_SON:Texas_S-PWSON-N10_ThermalVias -> Package_SON:Texas_S-PVSON-N10_ThermalVias
Changed lines of the file:
@@
 P 1400 2100
 F 0 "BT1" H 1518 2196 50  0000 L CNN
-F 1 "Li-Po 3.7V 800mAh" H 1518 2105 50  0000 L CNN
-F 2 "Connector_JST:JST_XH_S02B-XH-A-1_1x02_P2.50mm_Horizontal" V 1400 2160 50  0001 C CNN
+F 1 "Li-Po" H 1518 2105 50  0000 L CNN
+F 2 "Connector_JST:JST_EH_S02B-EH_1x02_P2.50mm_Horizontal" V 1400 2160 50  0001 C CNN
 F 3 "~" V 1400 2160 50  0001 C CNN
 	1    1400 2100
@@
 F 0 "U1" H 3100 2417 50  0000 C CNN
 F 1 "TPS63002" H 3100 2326 50  0000 C CNN
-F 2 "Package_SON:Texas_S-PWSON-N10_ThermalVias" H 3100 1100 50  0001 C CNN
+F 2 "Package_SON:Texas_S-PVSON-N10_ThermalVias" H 3100 1100 50  0001 C CNN
 F 3 "https://strawberry-linux.com/pub/tps63000.pdf" H 3100 1750 50  0001 C CNN
 F 4 "661-7061" H 0   0   50  0001 C CNN "品番"
@@
 L Connector_Generic:Conn_02x03_Odd_Even J5
 U 1 1 5C395DCA
-P 4950 4150
-F 0 "J5" H 5000 4467 50  0000 C CNN
-F 1 "IMU_Board" H 5000 4376 50  0000 C CNN
-F 2 "Connector_PinHeader_1.27mm:PinHeader_2x05_P1.27mm_Vertical" H 4950 4150 50  0001 C CNN
-F 3 "~" H 4950 4150 50  0001 C CNN
-F 4 "秋月" H 4950 4150 50  0001 C CNN "購入先"
-F 5 "C-13806" H 4950 4150 50  0001 C CNN "品番"
-	1    4950 4150
-	1    0    0    -1
+P 5050 4150
+F 0 "J5" H 5100 4467 50  0000 C CNN
+F 1 "IMU_Board" H 5100 4376 50  0000 C CNN
+F 2 "Connector_PinHeader_1.27mm:PinHeader_2x05_P1.27mm_Vertical" H 5050 4150 50  0001 C CNN
+F 3 "~" H 5050 4150 50  0001 C CNN
+F 4 "秋月" H 5050 4150 50  0001 C CNN "購入先"
+F 5 "C-13806" H 5050 4150 50  0001 C CNN "品番"
+	1    5050 4150
+	-1   0    0    -1
 $EndComp
 $Comp
@@
 F 0 "J2" H 4720 2025 50  0000 C CNN
 F 1 "IMU_Power" H 4720 2116 50  0000 C CNN
-F 2 "Connector_JST:JST_XH_S02B-XH-A_1x02_P2.50mm_Horizontal" H 4800 2350 50  0001 C CNN
+F 2 "Connector_JST:JST_EH_B02B-EH-A_1x02_P2.50mm_Vertical" H 4800 2350 50  0001 C CNN
 F 3 "~" H 4800 2350 50  0001 C CNN
 F 4 "C-12262" H 0   0   50  0001 C CNN "品番"
@@
 F 0 "J4" H 4329 3542 50  0000 L CNN
 F 1 "flight_pin" H 4329 3451 50  0000 L CNN
-F 2 "Connector_JST:JST_XH_S02B-XH-A-1_1x02_P2.50mm_Horizontal" H 4250 3550 50  0001 C CNN
+F 2 "Connector_JST:JST_EH_S02B-EH_1x02_P2.50mm_Horizontal" H 4250 3550 50  0001 C CNN
 F 3 "~" H 4250 3550 50  0001 C CNN
 F 4 "C-12262" H 0   0   50  0001 C CNN "品番"
@@
 F 0 "J7" H 4950 5350 50  0000 C CNN
 F 1 "LED_Board" H 4750 5250 50  0000 C CNN
-F 2 "Connector_JST:JST_XH_S04B-XH-A_1x04_P2.50mm_Horizontal" H 4950 5050 50  0001 C CNN
+F 2 "Connector_JST:JST_EH_S04B-EH_1x04_P2.50mm_Horizontal" H 4950 5050 50  0001 C CNN
 F 3 "~" H 4950 5050 50  0001 C CNN
 F 4 "C-12842" H 0   0   50  0001 C CNN "品番"
@@
 F 0 "J1" H 720 2217 50  0000 C CNN
 F 1 "Charge" H 720 2126 50  0000 C CNN
-F 2 "Connector_JST:JST_XH_S02B-XH-A_1x02_P2.50mm_Horizontal" H 800 2000 50  0001 C CNN
+F 2 "Connector_JST:JST_EH_S02B-EH_1x02_P2.50mm_Horizontal" H 800 2000 50  0001 C CNN
 F 3 "~" H 800 2000 50  0001 C CNN
 F 4 "C-12262" H 0   0   50  0001 C CNN "品番"
