File: PCB/EDAMAME_carrier_v3/EDAMAME_carrier_v3.kicad_pcb (KiCad board)
At the start: 2 copper layers, 180 x 100 mm, 73 parts, among them J1 POWER, J10 LED_T, J11 LED_B, J12 IN, J13 OUT, J2 DATA, J3 STlink, J4 LED_L, J5 LED_L, J6 LED_R, J7 LED_T, J8 LED_B, J9 LED_R, U1 STM32F042F6Px, U2 XC6202P332PR-G, U3 TPS63001

Commit message: Add PCB layout
Parts:
- removed C4: 10u, Capacitor_SMD:C_0805_2012Metric_Pad1.15x1.40mm_HandSolder
- removed C5: 1u, Capacitor_SMD:C_0805_2012Metric_Pad1.15x1.40mm_HandSolder
- removed C6, C7: 0.1u, Capacitor_SMD:C_0603_1608Metric_Pad1.05x0.95mm_HandSolder
- removed D10, D11, D12, D13, D14, D15, D16, D17, D18, D19, D20, D21, D22, D23, D24, D25, D26, D27, D28, D29, D30, D31, D32, D33, D34, D35, D36, D37, D38, D39, D4, D40, D41, D42, D43, D44, D45, D46, D47, D48, D5, D6, D7, D8, D9: S6812Side, user:S6812Side_top
- removed J10: LED_T, LED_Frame:LED_socket
- removed J11: LED_B, LED_Frame:LED_socket
- removed J12: IN, Connector_JST:JST_EH_S02B-EH_1x02_P2.50mm_Horizontal
- removed J13: OUT, Connector_JST:JST_EH_S02B-EH_1x02_P2.50mm_Horizontal
- removed J8: LED_B, LED_Frame:LED_Frame
- removed J9: LED_R, LED_Frame:LED_socket
- removed JP1: EN, Jumper:SolderJumper-2_P1.3mm_Open_Pad1.0x1.5mm
- removed L1: 2.2uH VLF4012-2R2, user:inductor_VLF4012-2R2
- removed U3: TPS63001, Package_SON:Texas_S-PVSON-N10_ThermalVias
- added BT1: Li-Po, Connector_JST:JST_EH_S02B-EH_1x02_P2.50mm_Horizontal, F.Cu at (69.5, 91.5)
- added BT2: Li-Po, Connector_JST:JST_EH_S02B-EH_1x02_P2.50mm_Horizontal, F.Cu at (78.0, 91.5)
- added BZ1: Buzzer, Capacitor_THT:CP_Radial_Tantal_D10.5mm_P5.00mm, F.Cu at (77.5, 134.5)
- added D101: LED_Small, LED_SMD:LED_0603_1608Metric_Pad1.05x0.95mm_HandSolder, F.Cu at (67.9, 66.5)
- added D102: LED_Small, LED_SMD:LED_0603_1608Metric_Pad1.05x0.95mm_HandSolder, F.Cu at (97.9, 66.5)
- added D103: LED_Small, LED_SMD:LED_0603_1608Metric_Pad1.05x0.95mm_HandSolder, F.Cu at (127.9, 66.5)
- added D104: LED_Small, LED_SMD:LED_0603_1608Metric_Pad1.05x0.95mm_HandSolder, F.Cu at (127.9, 104.0)
- added J101: Nichrome1, Connector_JST:JST_EH_S02B-EH_1x02_P2.50mm_Horizontal, F.Cu at (60.0, 60.0)
- added J102: Nichrome2, Connector_JST:JST_EH_S02B-EH_1x02_P2.50mm_Horizontal, F.Cu at (90.0, 60.0)
- added J103: Nichrome3, Connector_JST:JST_EH_S02B-EH_1x02_P2.50mm_Horizontal, F.Cu at (120.0, 60.0)
- added J104: Nichrome4, Connector_JST:JST_EH_S02B-EH_1x02_P2.50mm_Horizontal, F.Cu at (120.0, 97.5)
- added Q1: NDS9936, Package_SO:SO-8_5.3x6.2mm_P1.27mm, B.Cu at (66.2, 109.0)
- added Q2: NDS9936, Package_SO:SO-8_5.3x6.2mm_P1.27mm, B.Cu at (83.8, 109.0)
- added R1: 1k, Resistor_SMD:R_0603_1608Metric_Pad1.05x0.95mm_HandSolder, F.Cu at (78.2, 110.4)
- added R101: 1k, Resistor_SMD:R_0603_1608Metric_Pad1.05x0.95mm_HandSolder, F.Cu at (67.9, 51.5)
- added R102: 1k, Resistor_SMD:R_0603_1608Metric_Pad1.05x0.95mm_HandSolder, F.Cu at (97.9, 51.5)
- added R103: 1k, Resistor_SMD:R_0603_1608Metric_Pad1.05x0.95mm_HandSolder, F.Cu at (127.9, 51.5)
- added R104: 1k, Resistor_SMD:R_0603_1608Metric_Pad1.05x0.95mm_HandSolder, F.Cu at (127.9, 89.0)
- added R2: 1k, Resistor_SMD:R_0603_1608Metric_Pad1.05x0.95mm_HandSolder, B.Cu at (81.1, 123.4)
- added R3: 1k, Resistor_SMD:R_0603_1608Metric_Pad1.05x0.95mm_HandSolder, B.Cu at (68.9, 123.5)
- added R4: 1k, Resistor_SMD:R_0603_1608Metric_Pad1.05x0.95mm_HandSolder, F.Cu at (64.5, 108.0)
- added R5: 1k, Resistor_SMD:R_0603_1608Metric_Pad1.05x0.95mm_HandSolder, F.Cu at (85.3, 108.3)
- added R6: 1k, Resistor_SMD:R_0603_1608Metric_Pad1.05x0.95mm_HandSolder, F.Cu at (63.6, 110.8)
- added R7: 1k, Resistor_SMD:R_0603_1608Metric_Pad1.05x0.95mm_HandSolder, F.Cu at (86.2, 110.8)
- added SW1: power, user:SS-12D01-VG4, F.Cu at (70.2, 103.0)
- added SW2: Delay_0, Package_DIP:DIP-10_W7.62mm_LongPads, F.Cu at (95.5, 126.0)
- added SW3: Delay_0, Package_DIP:DIP-10_W7.62mm_LongPads, F.Cu at (62.1, 126.0)
- added T101: Nichrome1, TerminalBlock_MetzConnect:TerminalBlock_MetzConnect_Type101_RT01602HBWC_1x02_P5.08mm_Horizontal, F.Cu at (67.0, 61.5)
- added T102: Nichrome2, TerminalBlock_MetzConnect:TerminalBlock_MetzConnect_Type101_RT01602HBWC_1x02_P5.08mm_Horizontal, F.Cu at (97.0, 61.5)
- added T103: Nichrome3, TerminalBlock_MetzConnect:TerminalBlock_MetzConnect_Type101_RT01602HBWC_1x02_P5.08mm_Horizontal, F.Cu at (127.0, 61.5)
- added T104: Nichrome4, TerminalBlock_MetzConnect:TerminalBlock_MetzConnect_Type101_RT01602HBWC_1x02_P5.08mm_Horizontal, F.Cu at (127.0, 99.0)
- C1: value 10u -> 0.1u; footprint Capacitor_SMD:C_0805_2012Metric_Pad1.15x1.40mm_HandSolder -> Capacitor_SMD:C_0603_1608Metric_Pad1.05x0.95mm_HandSolder; moved to B.Cu
- D1, D2, D3: value S6812Side -> LED_Small; footprint user:S6812Side_top -> LED_SMD:LED_0603_1608Metric_Pad1.05x0.95mm_HandSolder
- J1: value POWER -> Charge; footprint Connector_JST:JST_EH_S02B-EH_1x02_P2.50mm_Horizontal -> Connector_JST:JST_EH_B03B-EH-A_1x03_P2.50mm_Vertical
- J2: value DATA -> Debug; footprint Connector_JST:JST_EH_S03B-EH_1x03_P2.50mm_Horizontal -> user:STlink
- J3: value STlink -> flightpin; footprint user:STlink -> Connector_JST:JST_EH_S02B-EH_1x02_P2.50mm_Horizontal
- J4: value LED_L -> Nichrome1; footprint LED_Frame:LED_Frame -> Connector_JST:JST_EH_S02B-EH_1x02_P2.50mm_Horizontal
- J5: value LED_L -> Nichrome2; footprint LED_Frame:LED_socket -> Connector_JST:JST_EH_S02B-EH_1x02_P2.50mm_Horizontal
- J6: value LED_R -> Nichrome3; footprint LED_Frame:LED_Frame -> Connector_JST:JST_EH_S02B-EH_1x02_P2.50mm_Horizontal
- J7: value LED_T -> Nichrome4; footprint LED_Frame:LED_Frame -> Connector_JST:JST_EH_S02B-EH_1x02_P2.50mm_Horizontal
- U1: moved to B.Cu
- U2: value XC6202P332PR-G -> NJM2391DL1-33; footprint Package_TO_SOT_SMD:SOT-89-3 -> Package_TO_SOT_SMD:TO-252-2
- moved D2 218.3 mm to (62.8, 108.0), turned to 90 degrees
- moved J4 203.5 mm to (60.0, 100.0), turned to 90 degrees
- moved D3 190.4 mm to (87.1, 108.3), turned to 90 degrees
- moved D1 187.0 mm to (76.5, 110.4), turned to 270 degrees
- moved J6 172.7 mm to (90.0, 106.0), turned to 270 degrees
- moved J7 152.8 mm to (90.0, 97.5)
- moved C3 81.2 mm to (82.5, 107.5), turned to 180 degrees
- moved J1 41.8 mm to (69.5, 97.0)
- moved J3 40.7 mm to (69.5, 134.0), turned to 180 degrees
- moved U2 34.7 mm to (81.5, 100.6), turned to 90 degrees
- moved J2 32.8 mm to (65.5, 129.0)
- moved C2 24.9 mm to (78.6, 107.5), turned to 0 degrees
- moved J5 24.2 mm to (60.0, 108.5)
- moved C1 15.7 mm to (75.0, 116.9), turned to 0 degrees
- moved U1 14.7 mm to (75.0, 121.5), turned to 0 degrees
Connections:
- net /NRST renamed Net-(U1-Pad4)
- C2 pad 1: +3V3 -> +BATT
- C3 pad 1: Net-(C3-Pad1) -> +3V3
- C3 pad 2: GNDD -> GND
- D1 pad 1: Net-(D1-Pad1) -> GND
- D2 pad 1: Net-(D1-Pad3) -> GND
- D2 pad 2: Net-(D1-Pad2) -> Net-(D2-Pad2)
- D3 pad 1: Net-(D2-Pad3) -> GND
- D3 pad 2: Net-(D1-Pad2) -> Net-(D3-Pad2)
- J1 pad 1: +BATT -> Net-(BT1-Pad1)
- J1 pad 2: GND -> Net-(BT1-Pad2)
- J2 pad 1: /SCL -> Net-(J2-Pad1)
- J2 pad 2: /SDA -> Net-(J2-Pad2)
- J2 pad 3: GND -> /SWCLK
- J3 pad 1: /TX -> /Flight_SW
- J3 pad 2: /RX -> GND
- J4 pad 1: Net-(D1-Pad4) -> Net-(J4-Pad1)
- J4 pad 2: Net-(D1-Pad4) -> +BATT
- J5 pad 1: GND -> Net-(J5-Pad1)
- J5 pad 2: GND -> +BATT
- J6 pad 1: Net-(D13-Pad4) -> Net-(J6-Pad1)
- J6 pad 2: Net-(D13-Pad4) -> +BATT
- J7 pad 1: Net-(D25-Pad4) -> Net-(J7-Pad1)
- J7 pad 2: Net-(D25-Pad4) -> +BATT
- U1 pad 1: Net-(U1-Pad1) -> /Flight_SW
- U1 pad 10: Net-(U1-Pad10) -> /Delay0_0.25s
- U1 pad 11: Net-(U1-Pad11) -> /Delay1_0.5s
- U1 pad 12: Net-(U1-Pad12) -> /Delay1_1s
- U1 pad 13: Net-(U1-Pad13) -> /Delay1_2s
- U1 pad 14: Net-(U1-Pad14) -> /Buzzer
- U1 pad 17: /TX -> /PWM0
- U1 pad 18: /RX -> /PWM1
- U1 pad 19: /SWDIO -> /SWCLK
- U1 pad 2: /SDA -> /Delay2_1s
- U1 pad 20: /SWCLK -> /SWDIO
- U1 pad 3: /SCL -> /Delay2_0.5s
- U1 pad 6: /LED_0 -> /Delay0_4s
- U1 pad 7: /LED_1 -> /Delay0_2s
- U1 pad 8: /LED_2 -> /Delay0_1s
- U1 pad 9: /LED_3 -> /Delay0_0.5s
- U2 pad 1: +3V3 -> +BATT
- U2 pad 3: +BATT -> +3V3
Routing:
- net /LED_0: track 223.7 -> 0.00 mm, vias 8 -> 0
- net /LED_1: track 210.8 -> 0.00 mm, vias 8 -> 0
- net /LED_2: track 197.3 -> 0.00 mm, vias 8 -> 0
- net /LED_3: track 190.1 -> 0.00 mm, vias 7 -> 0
- net +BATT: track 267.4 -> 92.0 mm
- net /PWM0: track 0.00 -> 29.3 mm, vias 0 -> 2
- net /PWM1: track 0.00 -> 28.3 mm, vias 0 -> 2
- net /TX: track 27.9 -> 0.00 mm
- net /RX: track 27.5 -> 0.00 mm
- net GND: track 53.2 -> 26.7 mm, vias 8 -> 0
- net /Flight_SW: track 0.00 -> 19.9 mm
- net /SWDIO: track 29.4 -> 10.3 mm
- net /Delay2_1s: track 0.00 -> 16.8 mm, vias 0 -> 1
- net /SDA: track 16.3 -> 0.00 mm
- net /Delay2_0.5s: track 0.00 -> 16.0 mm, vias 0 -> 1
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- added copper zone on B.Cu, net Net-(J4-Pad1)
- added copper zone on B.Cu, net Net-(J5-Pad1)
- added copper zone on B.Cu, net Net-(J6-Pad1)
- added copper zone on B.Cu, net Net-(J7-Pad1)
Other:
- board size 180 x 100 mm -> 85 x 95 mm
- board text added: "+ -"
- board text added: ".25s 0.5s 1.0s 2.0s 4.0s"
- board text added: "0.5s 1.0s 2.0s 0.5s 1.0s"
- board text added: "1(F→A)"
- board text added: "2|4 (A|B)"
- board text added: "3 (A→B)"
- board text added: "A"
- board text added: "B"
- board text added: "F"
- board text added: "ON OFF"
- board text added: "SOMESAT EDAMAME Carrier V3.0 @n_yosihisa 2019/01/20"
