File: PCB/EDAMAME_carrier_v3/EDAMAME_carrier_v3.sch (KiCad schematic (older format))
At the start: 43 parts, among them J1 Charge, J10 Nichrome4, J11 Nichrome1, J12 Nichrome2, J13 Nichrome3, J14 Nichrome4, J2 flightpin, J3 Nichrome1, J4 Nichrome2, J5 Nichrome3, J6 Nichrome4, J7 Nichrome1, J8 Nichrome2, J9 Nichrome3, Q1 NDS9936, Q2 NDS9936, SW1 power, SW2 Delay_0, SW3 Delay_0, U1 STM32F042F6Px, U2 NJM2391DL1-33

Commit message: Add PCB layout
Parts:
- removed D1, D2, D3, D4: LED_Small, LED_SMD:LED_0603_1608Metric_Pad1.05x0.95mm_HandSolder, symbol Device:LED_Small
- removed J10: Nichrome4, Connector_JST:JST_EH_S02B-EH_1x02_P2.50mm_Horizontal, symbol Connector:Conn_01x02_Male
- removed J11: Nichrome1, TerminalBlock_MetzConnect:TerminalBlock_MetzConnect_Type101_RT01602HBWC_1x02_P5.08mm_Horizontal, symbol Connector:Screw_Terminal_01x02
- removed J12: Nichrome2, TerminalBlock_MetzConnect:TerminalBlock_MetzConnect_Type101_RT01602HBWC_1x02_P5.08mm_Horizontal, symbol Connector:Screw_Terminal_01x02
- removed J13: Nichrome3, TerminalBlock_MetzConnect:TerminalBlock_MetzConnect_Type101_RT01602HBWC_1x02_P5.08mm_Horizontal, symbol Connector:Screw_Terminal_01x02
- removed J14: Nichrome4, TerminalBlock_MetzConnect:TerminalBlock_MetzConnect_Type101_RT01602HBWC_1x02_P5.08mm_Horizontal, symbol Connector:Screw_Terminal_01x02
- removed J7: Nichrome1, Connector_JST:JST_EH_S02B-EH_1x02_P2.50mm_Horizontal, symbol Connector:Conn_01x02_Male
- removed J8: Nichrome2, Connector_JST:JST_EH_S02B-EH_1x02_P2.50mm_Horizontal, symbol Connector:Conn_01x02_Male
- removed J9: Nichrome3, Connector_JST:JST_EH_S02B-EH_1x02_P2.50mm_Horizontal, symbol Connector:Conn_01x02_Male
- removed R4, R5, R6: 1k, Resistor_SMD:R_0603_1608Metric_Pad1.05x0.95mm_HandSolder, symbol Device:R_Small
- added C1: 0.1u, Capacitor_SMD:C_0603_1608Metric_Pad1.05x0.95mm_HandSolder, symbol Device:C_Small
- added J2: Debug, user:STlink, symbol Connector_Generic:Conn_01x05
- BZ1: 購入先 (none) -> 秋月
- renumbered C1 to C2, C2 to C3, D5 to D1, D6 to D2, D7 to D3, J2 to J3, J3 to J4, J4 to J5, J5 to J6, J6 to J7, R7 to R1, R8 to R2, R9 to R4, R10 to R5, R1 to R6, R2 to R7
Connections:
- wire segments 144 -> 122
